File: pcb/musashi60.kicad_pcb (KiCad board)
At the start: 2 copper layers, 175 x 135.7 mm, 79 parts, among them J1 MJ-4PP-9, U1 ProMicro_r

Commit message: update pcb
Parts:
- moved D_F2 7.14 mm to (61.9, 56.0)
- moved D_D5 5.61 mm to (116.1, 117.9)
- moved D_F1 4.76 mm to (61.9, 36.9)
- moved SW_F2 4.76 mm to (61.9, 47.6)
- moved SW_F3 4.76 mm to (61.9, 66.7)
- moved SW_F1 4.76 mm to (61.9, 28.6)
- moved D_F3 4.76 mm to (61.9, 75.0)
- moved SW_F4 4.76 mm to (61.9, 85.7)
- moved D_F4 4.76 mm to (61.9, 94.1)
- moved D_B5 3.24 mm to (153.2, 127.6)
- moved D_C5 3.19 mm to (135.1, 121.4)
- moved D_A5 3.13 mm to (167.0, 141.3)
Other:
- outline, holes or cut-outs redrawn
Changed lines of the file:
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@@
     (38 B.Mask user hide)
     (39 F.Mask user hide)
-    (40 Dwgs.User user)
+    (40 Dwgs.User user hide)
     (41 Cmts.User user hide)
     (42 Eco1.User user)
-    (43 Eco2.User user hide)
+    (43 Eco2.User user)
     (44 Edge.Cuts user)
     (45 Margin user hide)
@@
   )
   (module foostan:D3_TH_SMD (layer F.Cu)
-    (at 170.099861 141.003579 300)
+    (at 166.99133 141.338405 300)
     (descr "Resitance 3 pas")
     (tags R)
@@
   )
   (module foostan:D3_TH_SMD (layer F.Cu)
-    (at 156.481704 127.556389 330)
+    (at 153.244705 127.556389 330)
     (descr "Resitance 3 pas")
     (tags R)
@@
   )
   (module foostan:D3_TH_SMD (layer F.Cu)
-    (at 138.1125 122.634375)
+    (at 135.14745 121.44426)
     (descr "Resitance 3 pas")
     (tags R)
@@
   )
   (module foostan:D3_TH_SMD (layer F.Cu)
-    (at 119.0625 122.634375)
+    (at 116.09737 117.87237)
     (descr "Resitance 3 pas")
     (tags R)
@@
   )
   (module foostan:D3_TH_SMD (layer F.Cu)
-    (at 61.9125 41.671875)
+    (at 61.9125 36.909355)
     (descr "Resitance 3 pas")
     (tags R)
@@
   )
   (module foostan:D3_TH_SMD (layer F.Cu)
-    (at 61.9125 63.103125)
+    (at 61.9125 55.95961)
     (descr "Resitance 3 pas")
     (tags R)
@@
   )
   (module foostan:D3_TH_SMD (layer F.Cu)
-    (at 61.9125 79.771875)
+    (at 61.91276 75.00969)
     (descr "Resitance 3 pas")
     (tags R)
@@
   )
   (module foostan:D3_TH_SMD (layer F.Cu)
-    (at 61.9125 98.821875)
+    (at 61.9125 94.05977)
     (descr "Resitance 3 pas")
     (tags R)
@@
   )
   (module foostan:CherryMX_Choc_Hotswap (layer F.Cu)
-    (at 61.9125 33.3375)
+    (at 61.9125 28.57512)
     (fp_text reference SW_F1 (at 7 8.1) (layer F.SilkS) hide
       (effects (font (size 1 1) (thickness 0.15)))
@@
   )
   (module foostan:CherryMX_Choc_Hotswap (layer F.Cu)
-    (at 61.9125 52.38772)
+    (at 61.9125 47.6252)
     (fp_text reference SW_F2 (at 7 8.1) (layer F.SilkS) hide
       (effects (font (size 1 1) (thickness 0.15)))
@@
   )
   (module foostan:CherryMX_Choc_Hotswap (layer F.Cu)
-    (at 61.9125 71.4375)
+    (at 61.9125 66.67498)
     (fp_text reference SW_F3 (at 7 8.1) (layer F.SilkS) hide
       (effects (font (size 1 1) (thickness 0.15)))
@@
   )
   (module foostan:CherryMX_Choc_Hotswap (layer F.Cu)
-    (at 61.9125 90.4875)
+    (at 61.91276 85.72536)
     (fp_text reference SW_F4 (at 7 8.1) (layer F.SilkS) hide
       (effects (font (size 1 1) (thickness 0.15)))
@@
       ))
   )
-  (gr_line (start 52.38772 104.77544) (end 78.58158 104.77544) (layer Edge.Cuts) (width 0.05))
+  (gr_line (start 52.38772 114.30048) (end 98.82229 114.30048) (layer Edge.Cuts) (width 0.05))
   (gr_text Musashi60 (at 89.29725 97.63166) (layer B.SilkS)
     (effects (font (size 4 4) (thickness 0.4)) (justify mirror))
@@
   (gr_line (start 147.6375 104.775) (end 166.6875 104.775) (layer Eco1.User) (width 0.15))
   (gr_line (start 144.607744 123.993524) (end 149.538247 105.592637) (layer Eco1.User) (width 0.15))
-  (gr_line (start 52.38772 128.58804) (end 52.38772 104.77544) (layer Edge.Cuts) (width 0.05))
-  (gr_line (start 169.06875 150.01875) (end 78.58158 104.77544) (layer Edge.Cuts) (width 0.05))
+  (gr_line (start 52.38772 128.58804) (end 52.38772 114.30048) (layer Edge.Cuts) (width 0.05))
+  (gr_line (start 169.06875 150.01875) (end 98.82229 114.30048) (layer Edge.Cuts) (width 0.05))
   (gr_line (start 169.06875 150.01875) (end 189.31017 150.01938) (layer Edge.Cuts) (width 0.05))
   (gr_line (start 52.38772 128.5875) (end 14.2875 128.5875) (layer Edge.Cuts) (width 0.05))
@@
   (gr_line (start 128.5875 19.05) (end 128.5875 23.8125) (layer Eco1.User) (width 0.15))
   (gr_line (start 109.5375 14.2875) (end 109.5375 19.05) (layer Eco1.User) (width 0.15))
-  (gr_line (start 71.4375 100.0125) (end 71.4375 90.4875) (layer Eco1.User) (width 0.15))
+  (gr_line (start 71.4375 95.2504) (end 71.4375 90.4875) (layer Eco1.User) (width 0.15))
   (gr_line (start 52.3875 123.825) (end 52.3875 100.0125) (layer Eco1.User) (width 0.15))
   (gr_line (start 33.3375 123.825) (end 52.3875 123.825) (layer Eco1.User) (width 0.15))
@@
   (gr_line (start 33.3375 85.725) (end 52.3875 85.725) (layer Eco1.User) (width 0.15))
   (gr_line (start 33.3375 104.775) (end 52.3875 104.775) (layer Eco1.User) (width 0.15))
-  (gr_line (start 52.3875 61.9125) (end 71.4375 61.9125) (layer Eco1.User) (width 0.15))
-  (gr_line (start 52.3875 42.8625) (end 71.4375 42.8625) (layer Eco1.User) (width 0.15))
+  (gr_line (start 52.3875 57.14998) (end 71.4375 57.14998) (layer Eco1.User) (width 0.15))
+  (gr_line (start 52.3875 38.09998) (end 71.4375 38.09998) (layer Eco1.User) (width 0.15))
   (gr_line (start 52.3875 42.8625) (end 52.3875 61.9125) (layer Eco1.User) (width 0.15))
-  (gr_line (start 52.3875 100.0125) (end 71.4375 100.0125) (layer Eco1.User) (width 0.15))
+  (gr_line (start 52.3875 95.24998) (end 71.4375 95.24998) (layer Eco1.User) (width 0.15))
   (gr_line (start 52.3875 80.9625) (end 52.3875 100.0125) (layer Eco1.User) (width 0.15))
   (gr_line (start 52.3875 61.9125) (end 52.3875 80.9625) (layer Eco1.User) (width 0.15))
-  (gr_line (start 52.3875 80.9625) (end 71.4375 80.9625) (layer Eco1.User) (width 0.15))
-  (gr_line (start 71.4375 23.8125) (end 52.3875 23.8125) (layer Eco1.User) (width 0.15))
-  (gr_line (start 52.3875 23.8125) (end 52.3875 42.8625) (layer Eco1.User) (width 0.15))
+  (gr_line (start 52.3875 76.19998) (end 71.4375 76.19998) (layer Eco1.User) (width 0.15))
+  (gr_line (start 71.4375 19.04998) (end 52.3875 19.04998) (layer Eco1.User) (width 0.15))
+  (gr_line (start 52.3875 19.05008) (end 52.3875 42.8625) (layer Eco1.User) (width 0.15))
   (gr_line (start 71.4375 52.3875) (end 90.4875 52.3875) (layer Eco1.User) (width 0.15))
   (gr_line (start 71.4375 33.3375) (end 90.4875 33.3375) (layer Eco1.User) (width 0.15))

Commit message: update pcb
Parts:
- moved D_C5 1.21 mm to (135.7, 120.4), turned to 345 degrees
Other:
- outline, holes or cut-outs redrawn

Commit message: update pcb
Parts:
- moved J1 7.99 mm to (158.4, 45.2), turned to 330 degrees
- moved SW_RST1 3.89 mm to (20.2, 46.4)
- moved H_F5 2.38 mm to (38.1, 17.9)
- moved H_D2 2.38 mm to (33.3, 17.9)
- moved H_D3 2.38 mm to (31.0, 17.9)
- moved H_F4 2.38 mm to (35.7, 17.9)
- moved H_GND1 2.38 mm to (40.5, 17.9)
- moved H_VCC1 2.38 mm to (28.6, 17.9)
- moved JP_LEFT 1.36 mm to (22.1, 17.9), turned to 180 degrees
- moved JP_RIGHT 1.19 mm to (19.1, 17.9), turned to 0 degrees
- renumbered JP_LEFT1 to JP_LEFT, JP_RIGHT1 to JP_RIGHT
Other:
- outline, holes or cut-outs redrawn
Changed lines of the file:
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@@
   (layers
     (0 F.Cu signal)
-    (31 B.Cu signal hide)
+    (31 B.Cu signal)
     (32 B.Adhes user hide)
     (33 F.Adhes user hide)
     (34 B.Paste user hide)
     (35 F.Paste user hide)
-    (36 B.SilkS user hide)
-    (37 F.SilkS user hide)
+    (36 B.SilkS user)
+    (37 F.SilkS user)
     (38 B.Mask user hide)
     (39 F.Mask user hide)
@@
   )
   (module foostan:MJ-4PP-9 (layer F.Cu)
-    (at 154.7819 52.38772)
-    (fp_text reference J1 (at -0.85 4.95) (layer F.Fab)
+    (at 158.35379 45.24394 330)
+    (fp_text reference J1 (at -0.85 4.95 150) (layer F.Fab)
       (effects (font (size 1 1) (thickness 0.15)))
     )
-    (fp_text value MJ-4PP-9 (at 0 14) (layer F.Fab) hide
+    (fp_text value MJ-4PP-9 (at 0 14 150) (layer F.Fab) hide
       (effects (font (size 1 1) (thickness 0.15)))
     )
@@
     (fp_line (start 3 12) (end -3 12) (layer F.SilkS) (width 0.15))
     (fp_line (start -3 12) (end -3 0) (layer F.SilkS) (width 0.15))
-    (fp_text user TRRS (at -0.8255 6.4135) (layer B.SilkS)
+    (fp_text user TRRS (at -0.8255 6.4135 150) (layer B.SilkS)
       (effects (font (size 1 1) (thickness 0.15)) (justify mirror))
     )
-    (fp_text user TRRS (at -0.75 6.45) (layer F.SilkS)
+    (fp_text user TRRS (at -0.75 6.45 150) (layer F.SilkS)
       (effects (font (size 1 1) (thickness 0.15)))
     )
-    (pad "" np_thru_hole circle (at -1.75 8.5) (size 1.2 1.2) (drill 1.2) (layers *.Cu *.Mask F.SilkS))
-    (pad "" np_thru_hole circle (at -1.75 1.5) (size 1.2 1.2) (drill 1.2) (layers *.Cu *.Mask F.SilkS))
-    (pad D thru_hole oval (at -3.85 10.3) (size 1.7 2.5) (drill oval 1 1.5) (layers *.Cu *.Mask F.SilkS)
+    (pad "" np_thru_hole circle (at -1.75 8.5 330) (size 1.2 1.2) (drill 1.2) (layers *.Cu *.Mask F.SilkS))
+    (pad "" np_thru_hole circle (at -1.75 1.5 330) (size 1.2 1.2) (drill 1.2) (layers *.Cu *.Mask F.SilkS))
+    (pad D thru_hole oval (at -3.85 10.3 330) (size 1.7 2.5) (drill oval 1 1.5) (layers *.Cu *.Mask F.SilkS)
       (net 16 VCC) (clearance 0.15))
-    (pad A thru_hole oval (at 0.35 11.8) (size 1.7 2.5) (drill oval 1 1.5) (layers *.Cu *.Mask F.SilkS)
+    (pad A thru_hole oval (at 0.35 11.8 330) (size 1.7 2.5) (drill oval 1 1.5) (layers *.Cu *.Mask F.SilkS)
       (net 56 "Net-(J1-PadA)") (clearance 0.15))
-    (pad B thru_hole oval (at -3.85 3.3) (size 1.7 2.5) (drill oval 1 1.5) (layers *.Cu *.Mask F.SilkS)
+    (pad B thru_hole oval (at -3.85 3.3 330) (size 1.7 2.5) (drill oval 1 1.5) (layers *.Cu *.Mask F.SilkS)
       (net 52 D2))
-    (pad C thru_hole oval (at -3.85 6.3) (size 1.7 2.5) (drill oval 1 1.5) (layers *.Cu *.Mask F.SilkS)
+    (pad C thru_hole oval (at -3.85 6.3 330) (size 1.7 2.5) (drill oval 1 1.5) (layers *.Cu *.Mask F.SilkS)
       (net 14 GND))
-    (pad "" np_thru_hole circle (at 0 1.5) (size 1.2 1.2) (drill 1.2) (layers *.Cu *.Mask F.SilkS))
-    (pad "" np_thru_hole circle (at 0 8.5) (size 1.2 1.2) (drill 1.2) (layers *.Cu *.Mask F.SilkS))
-    (pad B thru_hole oval (at 2.1 3.3) (size 1.7 2.5) (drill oval 1 1.5) (layers *.Cu *.Mask F.SilkS)
+    (pad "" np_thru_hole circle (at 0 1.5 330) (size 1.2 1.2) (drill 1.2) (layers *.Cu *.Mask F.SilkS))
+    (pad "" np_thru_hole circle (at 0 8.5 330) (size 1.2 1.2) (drill 1.2) (layers *.Cu *.Mask F.SilkS))
+    (pad B thru_hole oval (at 2.1 3.3 330) (size 1.7 2.5) (drill oval 1 1.5) (layers *.Cu *.Mask F.SilkS)
       (net 52 D2))
-    (pad C thru_hole oval (at 2.1 6.3) (size 1.7 2.5) (drill oval 1 1.5) (layers *.Cu *.Mask F.SilkS)
+    (pad C thru_hole oval (at 2.1 6.3 330) (size 1.7 2.5) (drill oval 1 1.5) (layers *.Cu *.Mask F.SilkS)
       (net 14 GND))
-    (pad D thru_hole oval (at 2.1 10.3) (size 1.7 2.5) (drill oval 1 1.5) (layers *.Cu *.Mask F.SilkS)
+    (pad D thru_hole oval (at 2.1 10.3 330) (size 1.7 2.5) (drill oval 1 1.5) (layers *.Cu *.Mask F.SilkS)
       (net 16 VCC) (clearance 0.15))
-    (pad A thru_hole oval (at -2.1 11.8) (size 1.7 2.5) (drill oval 1 1.5) (layers *.Cu *.Mask F.SilkS)
+    (pad A thru_hole oval (at -2.1 11.8 330) (size 1.7 2.5) (drill oval 1 1.5) (layers *.Cu *.Mask F.SilkS)
       (net 56 "Net-(J1-PadA)") (clearance 0.15))
     (model "../../../../../../Users/pluis/Documents/Magic Briefcase/Documents/KiCad/3d/AB2_TRS_3p5MM_PTH.wrl"
@@
   )
   (module foostan:ResetSW (layer F.Cu)
-    (at 24.13449 46.43457)
+    (at 20.24071 46.43457)
     (fp_text reference SW_RST1 (at 0 2.55) (layer F.SilkS) hide
       (effects (font (size 1 1) (thickness 0.15)))
@@
   )
   (module foostan:1pin_conn (layer F.Cu)
-    (at 30.95638 17.85945)
+    (at 33.33764 17.85945)
     (descr "Resitance 3 pas")
     (tags R)
@@
   )
   (module foostan:1pin_conn (layer F.Cu)
-    (at 28.57512 17.85945)
+    (at 30.95638 17.85945)
     (descr "Resitance 3 pas")
     (tags R)
@@
   )
   (module foostan:1pin_conn (layer F.Cu)
-    (at 33.33764 17.85945)
+    (at 35.7189 17.85945)
     (descr "Resitance 3 pas")
     (tags R)
@@
   )
   (module foostan:1pin_conn (layer F.Cu)
-    (at 35.7189 17.85945)
+    (at 38.10016 17.85945)
     (descr "Resitance 3 pas")
     (tags R)
@@
   )
   (module foostan:1pin_conn (layer F.Cu)
-    (at 38.10016 17.85945)
+    (at 40.48142 17.85945)
     (descr "Resitance 3 pas")
     (tags R)
@@
   )
   (module foostan:1pin_conn (layer F.Cu)
-    (at 26.19386 17.85945)
+    (at 28.57512 17.85945)
     (descr "Resitance 3 pas")
     (tags R)
@@
   )
   (module Jumper:SolderJumper-2_P1.3mm_Open_RoundedPad1.0x1.5mm (layer F.Cu)
-    (at 21.43134 19.05008 270)
+    (at 22.08134 17.85945 180)
     (descr "SMD Solder Jumper, 1x1.5mm, rounded Pads, 0.3mm gap, open")
     (tags "solder jumper open")
     (attr virtual)
-    (fp_text reference JP_LEFT1 (at 0 -1.8 90) (layer F.SilkS)
+    (fp_text reference JP_LEFT (at 0 -1.8) (layer F.SilkS)
       (effects (font (size 1 1) (thickness 0.15)))
     )
-    (fp_text value Jumper (at 0 1.9 90) (layer F.Fab)
+    (fp_text value Jumper (at 0 1.9) (layer F.Fab)
       (effects (font (size 1 1) (thickness 0.15)))
     )
@@
     (fp_arc (start -0.7 0.3) (end -1.4 0.3) (angle -90) (layer F.SilkS) (width 0.12))
     (fp_arc (start -0.7 -0.3) (end -0.7 -1) (angle -90) (layer F.SilkS) (width 0.12))
-    (pad 1 smd custom (at -0.65 0 270) (size 1 0.5) (layers F.Cu F.Mask)
+    (pad 1 smd custom (at -0.65 0 180) (size 1 0.5) (layers F.Cu F.Mask)
       (net 16 VCC) (zone_connect 2)
       (options (clearance outline) (anchor rect))
@@
            (xy 0 -0.75) (xy 0.5 -0.75) (xy 0.5 0.75) (xy 0 0.75)) (width 0))
       ))
-    (pad 2 smd custom (at 0.65 0 270) (size 1 0.5) (layers F.Cu F.Mask)
+    (pad 2 smd custom (at 0.65 0 180) (size 1 0.5) (layers F.Cu F.Mask)
       (net 57 B6) (zone_connect 2)
       (options (clearance outline) (anchor rect))
@@
   )
   (module Jumper:SolderJumper-2_P1.3mm_Open_RoundedPad1.0x1.5mm (layer B.Cu)
-    (at 19.05008 19.05008 270)
+    (at 19.05008 17.85945)
     (descr "SMD Solder Jumper, 1x1.5mm, rounded Pads, 0.3mm gap, open")
     (tags "solder jumper open")
     (attr virtual)
-    (fp_text reference JP_RIGHT1 (at 0 1.8 90) (layer B.SilkS)
+    (fp_text reference JP_RIGHT (at 0 1.8) (layer B.SilkS)
       (effects (font (size 1 1) (thickness 0.15)) (justify mirror))
     )
-    (fp_text value Jumper (at 0 -1.9 90) (layer B.Fab)
+    (fp_text value Jumper (at 0 -1.9) (layer B.Fab)
       (effects (font (size 1 1) (thickness 0.15)) (justify mirror))
     )
@@
     (fp_arc (start -0.7 -0.3) (end -1.4 -0.3) (angle 90) (layer B.SilkS) (width 0.12))
     (fp_arc (start -0.7 0.3) (end -0.7 1) (angle 90) (layer B.SilkS) (width 0.12))
-    (pad 1 smd custom (at -0.65 0 270) (size 1 0.5) (layers B.Cu B.Mask)
+    (pad 1 smd custom (at -0.65 0) (size 1 0.5) (layers B.Cu B.Mask)
       (net 14 GND) (zone_connect 2)
       (options (clearance outline) (anchor rect))
@@
            (xy 0 0.75) (xy 0.5 0.75) (xy 0.5 -0.75) (xy 0 -0.75)) (width 0))
       ))
-    (pad 2 smd custom (at 0.65 0 270) (size 1 0.5) (layers B.Cu B.Mask)
+    (pad 2 smd custom (at 0.65 0) (size 1 0.5) (layers B.Cu B.Mask)
       (net 57 B6) (zone_connect 2)
       (options (clearance outline) (anchor rect))
@@
   (gr_line (start 147.6375 104.775) (end 166.6875 104.775) (layer Eco1.User) (width 0.15))
   (gr_line (start 144.607744 123.993524) (end 149.538247 105.592637) (layer Eco1.User) (width 0.15))
-  (gr_line (start 170.26009 150.01938) (end 107.1567 128.58804) (layer Edge.Cuts) (width 0.05))
+  (gr_line (start 170.26009 150.01938) (end 109.53796 128.58804) (layer Edge.Cuts) (width 0.05))
   (gr_line (start 170.26009 150.01938) (end 189.31017 150.01938) (layer Edge.Cuts) (width 0.05))
-  (gr_line (start 107.1567 128.58804) (end 14.2875 128.5875) (layer Edge.Cuts) (width 0.05))
+  (gr_line (start 109.53796 128.58804) (end 14.2875 128.5875) (layer Edge.Cuts) (width 0.05))
   (gr_line (start 126.206393 119.062358) (end 144.60728 123.992861) (layer Eco1.User) (width 0.15))
   (gr_line (start 149.537783 105.591974) (end 131.136896 100.661471) (layer Eco1.User) (width 0.15))

Commit message: update pcb
Parts:
- added G***: LOGO, local:musashi60-silk, B.Cu at (79.8, 108.3)
- added G***: LOGO, local:musashi60-silk, F.Cu at (79.8, 108.3)
Other:
- board text removed: "Musashi60"
