File: pcb/musashi60.kicad_pcb (KiCad board)
At the start: 2 copper layers, 175 x 135.7 mm, 81 parts, among them J1 MJ-4PP-9, U1 ProMicro_r

Commit message: update pcb
Parts:
- renumbered G*** to G_LOGO_B, G*** to G_LOGO_F

Commit message: update pcb
Parts:
- moved J1 3.37 mm to (156.0, 47.6), turned to 0 degrees
Other:
- outline, holes or cut-outs redrawn
Changed lines of the file:
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@@
   (general
     (thickness 1.6)
-    (drawings 102)
+    (drawings 106)
     (tracks 0)
     (zones 0)
@@
     (0 F.Cu signal)
     (31 B.Cu signal)
-    (32 B.Adhes user hide)
-    (33 F.Adhes user hide)
-    (34 B.Paste user hide)
-    (35 F.Paste user hide)
+    (32 B.Adhes user)
+    (33 F.Adhes user)
+    (34 B.Paste user)
+    (35 F.Paste user)
     (36 B.SilkS user)
     (37 F.SilkS user)
     (38 B.Mask user hide)
     (39 F.Mask user hide)
-    (40 Dwgs.User user)
+    (40 Dwgs.User user hide)
     (41 Cmts.User user hide)
-    (42 Eco1.User user)
+    (42 Eco1.User user hide)
     (43 Eco2.User user)
     (44 Edge.Cuts user)
@@
   )
   (module foostan:MJ-4PP-9 (layer F.Cu)
-    (at 158.35379 45.24394 330)
-    (fp_text reference J1 (at -0.85 4.95 150) (layer F.Fab)
+    (at 155.97253 47.6252)
+    (fp_text reference J1 (at -0.85 4.95) (layer F.Fab)
       (effects (font (size 1 1) (thickness 0.15)))
     )
-    (fp_text value MJ-4PP-9 (at 0 14 150) (layer F.Fab) hide
+    (fp_text value MJ-4PP-9 (at 0 14) (layer F.Fab) hide
       (effects (font (size 1 1) (thickness 0.15)))
     )
@@
     (fp_line (start 3 12) (end -3 12) (layer F.SilkS) (width 0.15))
     (fp_line (start -3 12) (end -3 0) (layer F.SilkS) (width 0.15))
-    (fp_text user TRRS (at -0.8255 6.4135 150) (layer B.SilkS)
+    (fp_text user TRRS (at -0.8255 6.4135) (layer B.SilkS)
       (effects (font (size 1 1) (thickness 0.15)) (justify mirror))
     )
-    (fp_text user TRRS (at -0.75 6.45 150) (layer F.SilkS)
+    (fp_text user TRRS (at -0.75 6.45) (layer F.SilkS)
       (effects (font (size 1 1) (thickness 0.15)))
     )
-    (pad "" np_thru_hole circle (at -1.75 8.5 330) (size 1.2 1.2) (drill 1.2) (layers *.Cu *.Mask F.SilkS))
-    (pad "" np_thru_hole circle (at -1.75 1.5 330) (size 1.2 1.2) (drill 1.2) (layers *.Cu *.Mask F.SilkS))
-    (pad D thru_hole oval (at -3.85 10.3 330) (size 1.7 2.5) (drill oval 1 1.5) (layers *.Cu *.Mask F.SilkS)
+    (pad "" np_thru_hole circle (at -1.75 8.5) (size 1.2 1.2) (drill 1.2) (layers *.Cu *.Mask F.SilkS))
+    (pad "" np_thru_hole circle (at -1.75 1.5) (size 1.2 1.2) (drill 1.2) (layers *.Cu *.Mask F.SilkS))
+    (pad D thru_hole oval (at -3.85 10.3) (size 1.7 2.5) (drill oval 1 1.5) (layers *.Cu *.Mask F.SilkS)
       (net 16 VCC) (clearance 0.15))
-    (pad A thru_hole oval (at 0.35 11.8 330) (size 1.7 2.5) (drill oval 1 1.5) (layers *.Cu *.Mask F.SilkS)
+    (pad A thru_hole oval (at 0.35 11.8) (size 1.7 2.5) (drill oval 1 1.5) (layers *.Cu *.Mask F.SilkS)
       (net 56 "Net-(J1-PadA)") (clearance 0.15))
-    (pad B thru_hole oval (at -3.85 3.3 330) (size 1.7 2.5) (drill oval 1 1.5) (layers *.Cu *.Mask F.SilkS)
+    (pad B thru_hole oval (at -3.85 3.3) (size 1.7 2.5) (drill oval 1 1.5) (layers *.Cu *.Mask F.SilkS)
       (net 52 D2))
-    (pad C thru_hole oval (at -3.85 6.3 330) (size 1.7 2.5) (drill oval 1 1.5) (layers *.Cu *.Mask F.SilkS)
+    (pad C thru_hole oval (at -3.85 6.3) (size 1.7 2.5) (drill oval 1 1.5) (layers *.Cu *.Mask F.SilkS)
       (net 14 GND))
-    (pad "" np_thru_hole circle (at 0 1.5 330) (size 1.2 1.2) (drill 1.2) (layers *.Cu *.Mask F.SilkS))
-    (pad "" np_thru_hole circle (at 0 8.5 330) (size 1.2 1.2) (drill 1.2) (layers *.Cu *.Mask F.SilkS))
-    (pad B thru_hole oval (at 2.1 3.3 330) (size 1.7 2.5) (drill oval 1 1.5) (layers *.Cu *.Mask F.SilkS)
+    (pad "" np_thru_hole circle (at 0 1.5) (size 1.2 1.2) (drill 1.2) (layers *.Cu *.Mask F.SilkS))
+    (pad "" np_thru_hole circle (at 0 8.5) (size 1.2 1.2) (drill 1.2) (layers *.Cu *.Mask F.SilkS))
+    (pad B thru_hole oval (at 2.1 3.3) (size 1.7 2.5) (drill oval 1 1.5) (layers *.Cu *.Mask F.SilkS)
       (net 52 D2))
-    (pad C thru_hole oval (at 2.1 6.3 330) (size 1.7 2.5) (drill oval 1 1.5) (layers *.Cu *.Mask F.SilkS)
+    (pad C thru_hole oval (at 2.1 6.3) (size 1.7 2.5) (drill oval 1 1.5) (layers *.Cu *.Mask F.SilkS)
       (net 14 GND))
-    (pad D thru_hole oval (at 2.1 10.3 330) (size 1.7 2.5) (drill oval 1 1.5) (layers *.Cu *.Mask F.SilkS)
+    (pad D thru_hole oval (at 2.1 10.3) (size 1.7 2.5) (drill oval 1 1.5) (layers *.Cu *.Mask F.SilkS)
       (net 16 VCC) (clearance 0.15))
-    (pad A thru_hole oval (at -2.1 11.8 330) (size 1.7 2.5) (drill oval 1 1.5) (layers *.Cu *.Mask F.SilkS)
+    (pad A thru_hole oval (at -2.1 11.8) (size 1.7 2.5) (drill oval 1 1.5) (layers *.Cu *.Mask F.SilkS)
       (net 56 "Net-(J1-PadA)") (clearance 0.15))
     (model "../../../../../../Users/pluis/Documents/Magic Briefcase/Documents/KiCad/3d/AB2_TRS_3p5MM_PTH.wrl"
@@
       ))
   )
+  (gr_line (start 33.33764 123.82552) (end 142.8756 123.82552) (layer Edge.Cuts) (width 0.05))
+  (gr_line (start 33.33764 128.58804) (end 33.33764 123.82552) (layer Edge.Cuts) (width 0.05))
+  (gr_line (start 147.63812 47.6252) (end 147.63812 14.28756) (layer Edge.Cuts) (width 0.05))
+  (gr_line (start 161.92568 47.6252) (end 147.63812 47.6252) (layer Edge.Cuts) (width 0.05))
   (dimension 175.02261 (width 0.15) (layer Dwgs.User)
     (gr_text "175.023 mm" (at 101.798865 158.46316) (layer Dwgs.User)
@@
   (gr_line (start 147.6375 104.775) (end 166.6875 104.775) (layer Eco1.User) (width 0.15))
   (gr_line (start 144.607744 123.993524) (end 149.538247 105.592637) (layer Eco1.User) (width 0.15))
-  (gr_line (start 170.26009 150.01938) (end 109.53796 128.58804) (layer Edge.Cuts) (width 0.05))
+  (gr_line (start 170.26009 150.01938) (end 142.8756 123.82552) (layer Edge.Cuts) (width 0.05))
   (gr_line (start 170.26009 150.01938) (end 189.31017 150.01938) (layer Edge.Cuts) (width 0.05))
-  (gr_line (start 109.53796 128.58804) (end 14.2875 128.5875) (layer Edge.Cuts) (width 0.05))
+  (gr_line (start 33.33764 128.58804) (end 14.2875 128.5875) (layer Edge.Cuts) (width 0.05))
   (gr_line (start 126.206393 119.062358) (end 144.60728 123.992861) (layer Eco1.User) (width 0.15))
   (gr_line (start 149.537783 105.591974) (end 131.136896 100.661471) (layer Eco1.User) (width 0.15))
@@
   (gr_line (start 33.3375 128.5875) (end 14.2875 128.5875) (layer Eco1.User) (width 0.15))
   (gr_line (start 33.3375 123.825) (end 33.3375 128.5875) (layer Eco1.User) (width 0.15))
-  (gr_line (start 152.40064 14.28756) (end 189.31017 150.01938) (layer Edge.Cuts) (width 0.05))
+  (gr_line (start 161.92568 47.6252) (end 189.31017 150.01938) (layer Edge.Cuts) (width 0.05))
   (dimension 135.73125 (width 0.15) (layer Dwgs.User)
     (gr_text "135.731 mm" (at -1.3 82.153125 270) (layer Dwgs.User)
@@
   )
   (gr_line (start 14.28756 14.28756) (end 14.2875 128.5875) (layer Edge.Cuts) (width 0.05))
-  (gr_line (start 14.28756 14.2875) (end 152.40064 14.28756) (layer Edge.Cuts) (width 0.05))
+  (gr_line (start 14.28756 14.2875) (end 147.63812 14.28756) (layer Edge.Cuts) (width 0.05))
   (gr_line (start 107.1567 100.01292) (end 107.1567 119.06292) (layer Eco1.User) (width 0.15))
   (gr_line (start 126.2067 100.01248) (end 107.1567 100.01248) (layer Eco1.User) (width 0.15))

Commit message: change clearance 0.2 -> 0.23
Other:
- net class Default: clearance 0.2 -> 0.23
- rule trace_clearance: 0.2 -> 0.23
