File: pcb/musashi60_wired.kicad_pcb (KiCad board)
At the start: 2 copper layers, 176.2 x 135.7 mm, 83 parts, among them J1 MJ-4PP-9, U1 ProMicro_r

Commit message: update wired pcb
Parts:
- removed HOLE1, HOLE2, HOLE3, HOLE4, HOLE5: MountingHole_3.2mm_M3, MountingHole:MountingHole_3.2mm_M3
- added G_LOGO_B: LOGO, local:musashi60-silk, B.Cu at (79.8, 108.3)
- added G_LOGO_F: LOGO, local:musashi60-silk, F.Cu at (79.8, 108.3)
- added JP_RIGHT: Jumper, Jumper:SolderJumper-2_P1.3mm_Open_RoundedPad1.0x1.5mm, B.Cu at (19.1, 17.9)
- moved SW_RST1 38.0 mm to (20.2, 46.4)
- moved D_G5 20.2 mm to (43.5, 122.6)
- moved SW_G2 19.6 mm to (42.9, 57.2)
- moved SW_G3 19.6 mm to (42.9, 76.2)
- moved D_G2 19.6 mm to (42.9, 65.5)
- moved D_G3 19.6 mm to (42.9, 84.5)
- moved D_G4 19.6 mm to (42.9, 103.6)
- moved SW_G5 19.6 mm to (42.9, 114.3)
- moved D_H4 19.6 mm to (23.8, 108.3)
- moved D_H5 19.6 mm to (23.8, 127.4)
- moved SW_H4 19.6 mm to (23.8, 100.0)
- moved SW_H5 19.6 mm to (23.8, 119.1)
- moved SW_G4 19.6 mm to (42.9, 95.3)
- moved D_H2 19.6 mm to (23.8, 70.2)
- moved D_H3 19.6 mm to (23.8, 89.3)
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- renumbered D2 to H_D2, D3 to H_D3, F4 to H_F4, F5 to H_F5, GND to H_GND1, VCC to H_VCC1, JP1 to JP_LEFT
Connections:
- JP_LEFT pad 1: GND -> VCC
Routing:
- net D4: track 336.2 -> 370.2 mm, vias 5 -> 6
- net D0: track 351.4 -> 378.3 mm, vias 6 -> 5
- net C6: track 340.7 -> 363.7 mm, vias 4 -> 5
- net B6: track 72.3 -> 51.6 mm, vias 1 -> 2
- net B5: track 226.1 -> 246.1 mm
- net B3: track 270.7 -> 251.3 mm
- net E6: track 236.8 -> 223.2 mm, vias 1 -> 2
- net F7: track 220.6 -> 208.5 mm, vias 2 -> 1
- net Net-(D_A3-Pad2): track 41.4 -> 30.5 mm, vias 0 -> 1
- net D2: track 189.8 -> 200.3 mm, vias 3 -> 1
- net B2: track 290.6 -> 301.0 mm, vias 1 -> 2
- net Net-(D_A4-Pad2): track 40.9 -> 30.6 mm, vias 0 -> 1
- net B1: track 252.6 -> 242.9 mm
- net RST: track 35.0 -> 25.6 mm
- net VCC: track 166.8 -> 175.3 mm
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Other:
- board size 176.2 x 135.7 mm -> 175 x 135.7 mm
- board text removed: "Musashi60"

Commit message: update wired pcb
Routing:
- net D4: track 370.2 -> 312.5 mm, vias 6 -> 5
- net B1: track 242.9 -> 297.2 mm, vias 3 -> 2
- net D7: track 229.5 -> 269.3 mm, vias 6 -> 2
- net D0: track 378.3 -> 415.1 mm, vias 5 -> 6
- net B2: track 301.0 -> 277.3 mm, vias 2 -> 0
- net E6: track 223.2 -> 242.6 mm
- net D1: track 312.9 -> 330.5 mm, vias 5 -> 3
- net B3: track 251.3 -> 268.0 mm
- net VCC: track 175.3 -> 190.8 mm, vias 0 -> 2
- net C6: track 363.7 -> 352.7 mm, vias 5 -> 6
- net Net-(D_H5-Pad2): track 41.2 -> 33.0 mm, vias 0 -> 1
- net Net-(D_B3-Pad2): track 47.3 -> 40.5 mm
- net Net-(D_C2-Pad2): track 46.6 -> 40.2 mm
- net GND: track 205.3 -> 199.2 mm, vias 0 -> 1
- net Net-(D_B5-Pad2): track 40.8 -> 34.7 mm
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Other:
- outline, holes or cut-outs redrawn
- net class Default: clearance 0.2 -> 0.23
- rule trace_clearance: 0.2 -> 0.23
