File: pcb/musashi60.sch (KiCad schematic (older format))
At the start: 78 parts, among them J1 MJ-4PP-9, U1 ProMicro_r

Commit message: add jumper for left hand
Parts:
- added JP_RIGHT1: Jumper, Jumper:SolderJumper-2_P1.3mm_Open_RoundedPad1.0x1.5mm, symbol Device:Jumper
- renumbered JP1 to JP_LEFT1
Connections:
- wire segments 101 -> 102
Changed lines of the file:
@@
 B6
 $Comp
-L Device:Jumper JP1
+L Device:Jumper JP_LEFT1
 U 1 1 5F738159
 P 1250 6400
-F 0 "JP1" H 1250 6268 50  0000 C CNN
+F 0 "JP_LEFT1" H 1250 6268 50  0000 C CNN
 F 1 "Jumper" H 1250 6177 50  0000 C CNN
 F 2 "Jumper:SolderJumper-2_P1.3mm_Open_RoundedPad1.0x1.5mm" H 1250 6400 50  0001 C CNN
 F 3 "~" H 1250 6400 50  0001 C CNN
 	1    1250 6400
-	1    0    0    -1
-$EndComp
-$Comp
-L power:GND #PWR02
-U 1 1 5F746B7E
-P 950 6400
-F 0 "#PWR02" H 950 6150 50  0001 C CNN
-F 1 "GND" H 955 6227 50  0000 C CNN
-F 2 "" H 950 6400 50  0001 C CNN
-F 3 "" H 950 6400 50  0001 C CNN
-	1    950  6400
 	1    0    0    -1
 $EndComp
@@
 	1    0    0    -1
 $EndComp
+$Comp
+L Device:Jumper JP_RIGHT1
+U 1 1 5F795429
+P 1250 6850
+F 0 "JP_RIGHT1" H 1250 6718 50  0000 C CNN
+F 1 "Jumper" H 1250 6627 50  0000 C CNN
+F 2 "Jumper:SolderJumper-2_P1.3mm_Open_RoundedPad1.0x1.5mm" H 1250 6850 50  0001 C CNN
+F 3 "~" H 1250 6850 50  0001 C CNN
+	1    1250 6850
+	1    0    0    -1
+$EndComp
+$Comp
+L power:GND #PWR05
+U 1 1 5F79542F
+P 950 6850
+F 0 "#PWR05" H 950 6600 50  0001 C CNN
+F 1 "GND" H 955 6677 50  0000 C CNN
+F 2 "" H 950 6850 50  0001 C CNN
+F 3 "" H 950 6850 50  0001 C CNN
+	1    950  6850
+	1    0    0    -1
+$EndComp
+$Comp
+L power:VCC #PWR02
+U 1 1 5F7A2499
+P 950 6400
+F 0 "#PWR02" H 950 6250 50  0001 C CNN
+F 1 "VCC" H 965 6573 50  0000 C CNN
+F 2 "" H 950 6400 50  0001 C CNN
+F 3 "" H 950 6400 50  0001 C CNN
+	1    950  6400
+	1    0    0    -1
+$EndComp
+Wire Wire Line
+	1550 6400 1550 6850
+Connection ~ 1550 6400
 $EndSCHEMATC

Commit message: update musashi60.sch
Parts:
- removed D_G5, D_H5: D, foostan:D3_TH_SMD, symbol Device:D
- removed SW_G5, SW_H5: SW_PUSH, foostan:CherryMX_Choc_Hotswap, symbol foostan:SW_PUSH
- SW_A3, SW_A4, SW_A5, SW_B1, SW_B2, SW_B3, SW_B4, SW_B5, SW_C1, SW_C2, SW_C3, SW_C4, SW_C5, SW_D1, SW_D2, SW_D3, SW_D4, SW_D5, SW_E1, SW_E2, SW_E3, SW_E4, SW_F1, SW_F2, SW_F3, SW_F4, SW_G2, SW_G3, SW_G4, SW_H2, SW_H3, SW_H4: footprint foostan:CherryMX_Choc_Hotswap -> local:CherryMX_Direct_Hotswap_Reversible
- renumbered H_D2 to D2, H_D3 to D3, H_F4 to F4, H_F5 to F5, H_GND1 to GND1, H_VCC1 to VCC1
Connections:
- wire segments 102 -> 98

Commit message: update circut
Parts:
- removed D_A3, D_H4: D, foostan:D3_TH_SMD, symbol Device:D
- removed SW_A3, SW_H4: SW_PUSH, local:CherryMX_Direct_Hotswap_Reversible, symbol foostan:SW_PUSH
- renumbered D_B1 to D_A1, D_B2 to D_A2, D_B3 to D_A3, D_B4 to D_A4, D_C1 to D_B1, D_C2 to D_B2, D_C3 to D_B3, D_C4 to D_B4, D_F1 to D_C1, D_H2 to D_C2, D_H3 to D_C3, D_G4 to D_C4, D_A4 to D_E5, D_F4 to D_F5, SW_B1 to SW_A1, SW_B2 to SW_A2, SW_B3 to SW_A3, SW_B4 to SW_A4, SW_C1 to SW_B1, SW_C2 to SW_B2, SW_C3 to SW_B3, SW_C4 to SW_B4, SW_F1 to SW_C1, SW_H2 to SW_C2, SW_H3 to SW_C3, SW_G4 to SW_C4, SW_A4 to SW_E5, SW_F4 to SW_F5
Connections:
- net labels removed: colH
- wire segments 98 -> 94
- no-connect marks 2 -> 3

Commit message: update for rev7 pcb
Parts:
- added B5: MountingHole_Pad, foostan:1pin_conn, symbol Mechanical:MountingHole_Pad
Connections:
- no-connect marks 3 -> 2
Changed lines of the file:
@@
 Text GLabel 1500 2900 0    50   Input ~ 0
 B3
-Text GLabel 2700 5000 0    50   Input ~ 0
+Text GLabel 2700 5200 0    50   Input ~ 0
 D1
-Text GLabel 3200 5000 2    50   Input ~ 0
+Text GLabel 3200 5200 2    50   Input ~ 0
 colA
 Wire Wire Line
-	2700 5000 3200 5000
-Text GLabel 2700 5200 0    50   Input ~ 0
+	2700 5200 3200 5200
+Text GLabel 2700 5400 0    50   Input ~ 0
 D0
-Text GLabel 3200 5200 2    50   Input ~ 0
+Text GLabel 3200 5400 2    50   Input ~ 0
 colB
 Wire Wire Line
-	2700 5200 3200 5200
+	2700 5400 3200 5400
 Text GLabel 1500 3000 0    50   Input ~ 0
 B2
@@
 	1    0    0    -1
 $EndComp
-Text GLabel 2700 5400 0    50   Input ~ 0
+Text GLabel 2700 5600 0    50   Input ~ 0
 D4
-Text GLabel 3200 5400 2    50   Input ~ 0
+Text GLabel 3200 5600 2    50   Input ~ 0
 colC
 Wire Wire Line
-	2700 5400 3200 5400
+	2700 5600 3200 5600
 Text GLabel 2900 2600 2    50   Input ~ 0
 D4
@@
 Text GLabel 4750 2150 0    50   Input ~ 0
 colG
-Text GLabel 2700 5600 0    50   Input ~ 0
+Text GLabel 2700 5800 0    50   Input ~ 0
 C6
-Text GLabel 3200 5600 2    50   Input ~ 0
+Text GLabel 3200 5800 2    50   Input ~ 0
 colD
-Wire Wire Line
-	2700 5600 3200 5600
-Text GLabel 2700 5800 0    50   Input ~ 0
-D7
-Text GLabel 3200 5800 2    50   Input ~ 0
-colE
 Wire Wire Line
 	2700 5800 3200 5800
 Text GLabel 2700 6000 0    50   Input ~ 0
+D7
+Text GLabel 3200 6000 2    50   Input ~ 0
+colE
+Wire Wire Line
+	2700 6000 3200 6000
+Text GLabel 2700 6200 0    50   Input ~ 0
 E6
-Text GLabel 3200 6000 2    50   Input ~ 0
+Text GLabel 3200 6200 2    50   Input ~ 0
 colF
 Wire Wire Line
-	2700 6000 3200 6000
+	2700 6200 3200 6200
 Text GLabel 2900 2700 2    50   Input ~ 0
 C6
@@
 Text GLabel 2900 3000 2    50   Input ~ 0
 B4
-Text GLabel 2700 6200 0    50   Input ~ 0
+Text GLabel 2700 6400 0    50   Input ~ 0
 B4
-Text GLabel 3200 6200 2    50   Input ~ 0
+Text GLabel 3200 6400 2    50   Input ~ 0
 colG
-Text GLabel 2700 6400 0    50   Input ~ 0
-B5
-Wire Wire Line
-	2700 6400 3200 6400
 Text GLabel 2900 3100 2    50   Input ~ 0
 B5
@@
 Text GLabel 1550 5400 0    50   Input ~ 0
 row1
-Text GLabel 5050 6550 0    50   Input ~ 0
+Text GLabel 5050 6350 0    50   Input ~ 0
 D3
-Text GLabel 2700 4800 0    50   Input ~ 0
+Text GLabel 2700 5000 0    50   Input ~ 0
 D2
-Text GLabel 3200 4800 2    50   Input ~ 0
+Text GLabel 3200 5000 2    50   Input ~ 0
 data
 Wire Wire Line
-	2700 4800 3200 4800
+	2700 5000 3200 5000
 Wire Wire Line
 	2050 6400 1550 6400
@@
 F7
 Wire Wire Line
-	5050 7150 5550 7150
-Wire Wire Line
 	5050 6950 5550 6950
+Wire Wire Line
+	5050 6750 5550 6750
+Text GLabel 5050 6750 0    50   Input ~ 0
+F4
 Text GLabel 5050 6950 0    50   Input ~ 0
-F4
-Text GLabel 5050 7150 0    50   Input ~ 0
 F5
 $Comp
 L Mechanical:MountingHole_Pad F4
 U 1 1 5F7D88A6
+P 5650 6750
+F 0 "F4" V 5696 6899 50  0000 L CNN
+F 1 "MountingHole_Pad" V 5605 6899 50  0000 L CNN
+F 2 "foostan:1pin_conn" H 5650 6750 50  0001 C CNN
+F 3 "~" H 5650 6750 50  0001 C CNN
+	1    5650 6750
+	0    1    -1   0
+$EndComp
+$Comp
+L Mechanical:MountingHole_Pad F5
+U 1 1 5F7DA890
 P 5650 6950
-F 0 "F4" V 5696 7099 50  0000 L CNN
+F 0 "F5" V 5696 7099 50  0000 L CNN
 F 1 "MountingHole_Pad" V 5605 7099 50  0000 L CNN
 F 2 "foostan:1pin_conn" H 5650 6950 50  0001 C CNN
@@
 	0    1    -1   0
 $EndComp
-$Comp
-L Mechanical:MountingHole_Pad F5
-U 1 1 5F7DA890
-P 5650 7150
-F 0 "F5" V 5696 7299 50  0000 L CNN
-F 1 "MountingHole_Pad" V 5605 7299 50  0000 L CNN
-F 2 "foostan:1pin_conn" H 5650 7150 50  0001 C CNN
-F 3 "~" H 5650 7150 50  0001 C CNN
-	1    5650 7150
-	0    1    -1   0
-$EndComp
-Wire Wire Line
-	2700 6200 3200 6200
-Wire Wire Line
-	5050 6550 5550 6550
+Wire Wire Line
+	2700 6400 3200 6400
+Wire Wire Line
+	5050 6350 5550 6350
 $Comp
 L Mechanical:MountingHole_Pad D3
 U 1 1 5F6F0153
-P 5650 6550
-F 0 "D3" V 5604 6700 50  0000 L CNN
-F 1 "MountingHole_Pad" V 5695 6700 50  0000 L CNN
-F 2 "foostan:1pin_conn" H 5650 6550 50  0001 C CNN
-F 3 "~" H 5650 6550 50  0001 C CNN
-	1    5650 6550
+P 5650 6350
+F 0 "D3" V 5604 6500 50  0000 L CNN
+F 1 "MountingHole_Pad" V 5695 6500 50  0000 L CNN
+F 2 "foostan:1pin_conn" H 5650 6350 50  0001 C CNN
+F 3 "~" H 5650 6350 50  0001 C CNN
+	1    5650 6350
 	0    1    1    0
 $EndComp
@@
 L Mechanical:MountingHole_Pad VCC1
 U 1 1 5F8B4206
-P 5650 6350
-F 0 "VCC1" V 5604 6500 50  0000 L CNN
-F 1 "MountingHole_Pad" V 5695 6500 50  0000 L CNN
-F 2 "foostan:1pin_conn" H 5650 6350 50  0001 C CNN
-F 3 "~" H 5650 6350 50  0001 C CNN
-	1    5650 6350
+P 5650 6150
+F 0 "VCC1" V 5604 6300 50  0000 L CNN
+F 1 "MountingHole_Pad" V 5695 6300 50  0000 L CNN
+F 2 "foostan:1pin_conn" H 5650 6150 50  0001 C CNN
+F 3 "~" H 5650 6150 50  0001 C CNN
+	1    5650 6150
 	0    1    1    0
 $EndComp
@@
 Text GLabel 3925 3875 2    50   Input ~ 0
 data
-Text GLabel 5050 6750 0    50   Input ~ 0
+Text GLabel 5050 6550 0    50   Input ~ 0
 D2
 Wire Wire Line
-	5050 6750 5550 6750
+	5050 6550 5550 6550
 $Comp
 L Mechanical:MountingHole_Pad D2
 U 1 1 5F900118
-P 5650 6750
-F 0 "D2" V 5604 6900 50  0000 L CNN
-F 1 "MountingHole_Pad" V 5695 6900 50  0000 L CNN
-F 2 "foostan:1pin_conn" H 5650 6750 50  0001 C CNN
-F 3 "~" H 5650 6750 50  0001 C CNN
-	1    5650 6750
+P 5650 6550
+F 0 "D2" V 5604 6700 50  0000 L CNN
+F 1 "MountingHole_Pad" V 5695 6700 50  0000 L CNN
+F 2 "foostan:1pin_conn" H 5650 6550 50  0001 C CNN
+F 3 "~" H 5650 6550 50  0001 C CNN
+	1    5650 6550
 	0    1    1    0
 $EndComp
 Wire Wire Line
-	5550 6350 5050 6350
+	5550 6150 5050 6150
 Wire Wire Line
 	5550 7350 5050 7350
@@
 L power:VCC #PWR03
 U 1 1 5F996DCC
-P 5050 6350
-F 0 "#PWR03" H 5050 6200 50  0001 C CNN
-F 1 "VCC" H 5065 6523 50  0000 C CNN
-F 2 "" H 5050 6350 50  0001 C CNN
-F 3 "" H 5050 6350 50  0001 C CNN
-	1    5050 6350
+P 5050 6150
+F 0 "#PWR03" H 5050 6000 50  0001 C CNN
+F 1 "VCC" H 5065 6323 50  0000 C CNN
+F 2 "" H 5050 6150 50  0001 C CNN
+F 3 "" H 5050 6150 50  0001 C CNN
+	1    5050 6150
 	1    0    0    -1
 $EndComp
@@
 Wire Wire Line
 	9550 2750 9650 2750
-NoConn ~ 3200 6400
 Wire Wire Line
 	4750 2150 4750 3100
@@
 Connection ~ 7450 2750
 Wire Wire Line
-	8150 3400 8150 3750
-Connection ~ 8150 3400
-Connection ~ 8150 3750
-Wire Wire Line
 	8150 4050 7450 4050
 Connection ~ 8150 4050
 Connection ~ 7450 4050
 Connection ~ 6750 5350
+Wire Wire Line
+	8150 3400 7450 3400
+Connection ~ 8150 3400
+Connection ~ 7450 3400
+Wire Wire Line
+	5050 7150 5550 7150
+Text GLabel 5050 7150 0    50   Input ~ 0
+B5
+$Comp
+L Mechanical:MountingHole_Pad B5
+U 1 1 6008F413
+P 5650 7150
+F 0 "B5" V 5696 7299 50  0000 L CNN
+F 1 "MountingHole_Pad" V 5605 7299 50  0000 L CNN
+F 2 "foostan:1pin_conn" H 5650 7150 50  0001 C CNN
+F 3 "~" H 5650 7150 50  0001 C CNN
+	1    5650 7150
+	0    1    -1   0
+$EndComp
 $EndSCHEMATC

Commit message: update circut for rev8
Parts:
- removed D_E5, D_F5, D_G2: D, foostan:D3_TH_SMD, symbol Device:D
- removed F4: MountingHole_Pad, foostan:1pin_conn, symbol Mechanical:MountingHole_Pad
- removed SW_E5, SW_F5, SW_G2: SW_PUSH, local:CherryMX_Direct_Hotswap_Reversible, symbol foostan:SW_PUSH
- added U2: joystick, local:J08K, symbol local:joystick
- renumbered F5 to B4, D_G3 to D_F2, D_F2 to D_F4, SW_G3 to SW_F2, SW_F2 to SW_F4
Connections:
- net labels removed: colG
- wire segments 94 -> 86
