File: pcb/musashi60.sch (KiCad schematic (older format))
At the start: 70 parts, among them J1 MJ-4PP-9, U1 ProMicro_r, U3 joystick_s

Commit message: use Joycon_Stick_Short
Parts:
- U3: footprint local:Joycon_Stick -> local:Joycon_Stick_Short
Changed lines of the file:
@@
 F 0 "U3" H 4778 3951 50  0000 L CNN
 F 1 "joystick_s" H 4778 3860 50  0000 L CNN
-F 2 "local:Joycon_Stick" H 4550 3600 50  0001 C CNN
+F 2 "local:Joycon_Stick_Short" H 4550 3600 50  0001 C CNN
 F 3 "" H 4550 3600 50  0001 C CNN
 	1    4550 3900

Commit message: remove test pin
Parts:
- removed B4, D2, D3, GND1, VCC1: MountingHole_Pad, foostan:1pin_conn, symbol Mechanical:MountingHole_Pad
Connections:
- wire segments 90 -> 85
Changed lines of the file:
@@
 Text GLabel 1550 5400 0    50   Input ~ 0
 row1
-Text GLabel 5050 6350 0    50   Input ~ 0
-D3
 Text GLabel 2700 5200 0    50   Input ~ 0
 D2
@@
 Text GLabel 2050 5600 2    50   Input ~ 0
 F7
-Wire Wire Line
-	5050 6750 5550 6750
-Text GLabel 5050 6750 0    50   Input ~ 0
-B4
-$Comp
-L Mechanical:MountingHole_Pad B4
-U 1 1 5F7DA890
-P 5650 6750
-F 0 "B4" V 5696 6899 50  0000 L CNN
-F 1 "MountingHole_Pad" V 5605 6899 50  0000 L CNN
-F 2 "foostan:1pin_conn" H 5650 6750 50  0001 C CNN
-F 3 "~" H 5650 6750 50  0001 C CNN
-	1    5650 6750
-	0    1    -1   0
-$EndComp
-Wire Wire Line
-	5050 6350 5550 6350
-$Comp
-L Mechanical:MountingHole_Pad D3
-U 1 1 5F6F0153
-P 5650 6350
-F 0 "D3" V 5604 6500 50  0000 L CNN
-F 1 "MountingHole_Pad" V 5695 6500 50  0000 L CNN
-F 2 "foostan:1pin_conn" H 5650 6350 50  0001 C CNN
-F 3 "~" H 5650 6350 50  0001 C CNN
-	1    5650 6350
-	0    1    1    0
-$EndComp
 Text GLabel 1500 2400 0    50   Input ~ 0
 F4
 Text GLabel 1500 2500 0    50   Input ~ 0
 F5
-$Comp
-L Mechanical:MountingHole_Pad GND1
-U 1 1 5F8A75FD
-P 5650 6950
-F 0 "GND1" V 5604 7100 50  0000 L CNN
-F 1 "MountingHole_Pad" V 5695 7100 50  0000 L CNN
-F 2 "foostan:1pin_conn" H 5650 6950 50  0001 C CNN
-F 3 "~" H 5650 6950 50  0001 C CNN
-	1    5650 6950
-	0    1    1    0
-$EndComp
-$Comp
-L Mechanical:MountingHole_Pad VCC1
-U 1 1 5F8B4206
-P 5650 6150
-F 0 "VCC1" V 5604 6300 50  0000 L CNN
-F 1 "MountingHole_Pad" V 5695 6300 50  0000 L CNN
-F 2 "foostan:1pin_conn" H 5650 6150 50  0001 C CNN
-F 3 "~" H 5650 6150 50  0001 C CNN
-	1    5650 6150
-	0    1    1    0
-$EndComp
 Wire Wire Line
 	2850 3975 3175 3975
 Text GLabel 3175 3975 2    50   Input ~ 0
 data
-Text GLabel 5050 6550 0    50   Input ~ 0
-D2
-Wire Wire Line
-	5050 6550 5550 6550
-$Comp
-L Mechanical:MountingHole_Pad D2
-U 1 1 5F900118
-P 5650 6550
-F 0 "D2" V 5604 6700 50  0000 L CNN
-F 1 "MountingHole_Pad" V 5695 6700 50  0000 L CNN
-F 2 "foostan:1pin_conn" H 5650 6550 50  0001 C CNN
-F 3 "~" H 5650 6550 50  0001 C CNN
-	1    5650 6550
-	0    1    1    0
-$EndComp
-Wire Wire Line
-	5550 6150 5050 6150
-Wire Wire Line
-	5550 6950 5050 6950
-$Comp
-L power:GND #PWR04
-U 1 1 5F995F04
-P 5050 6950
-F 0 "#PWR04" H 5050 6700 50  0001 C CNN
-F 1 "GND" H 5055 6777 50  0000 C CNN
-F 2 "" H 5050 6950 50  0001 C CNN
-F 3 "" H 5050 6950 50  0001 C CNN
-	1    5050 6950
-	1    0    0    -1
-$EndComp
-$Comp
-L power:VCC #PWR03
-U 1 1 5F996DCC
-P 5050 6150
-F 0 "#PWR03" H 5050 6000 50  0001 C CNN
-F 1 "VCC" H 5065 6323 50  0000 C CNN
-F 2 "" H 5050 6150 50  0001 C CNN
-F 3 "" H 5050 6150 50  0001 C CNN
-	1    5050 6150
-	1    0    0    -1
-$EndComp
 $Comp
 L Device:Jumper JP_RIGHT1

Commit message: update scheme
Parts:
- removed D_E5, D_F1: D, foostan:D3_TH_SMD, symbol Device:D
- removed JP_NOJS1: Jumper, Jumper:SolderJumper-2_P1.3mm_Open_RoundedPad1.0x1.5mm, symbol Device:Jumper
- removed SW_E5, SW_F1: SW_PUSH, local:CherryMX_Direct_Hotswap_Reversible, symbol foostan:SW_PUSH
- removed U3: joystick_s, local:Joycon_Stick_Short, symbol local:joystick_s
- added D_G2, D_G3: D, foostan:D3_TH_SMD, symbol Device:D
- added SW_G2, SW_G3: SW_PUSH, local:CherryMX_Direct_Hotswap_Reversible, symbol foostan:SW_PUSH
- renumbered D_A1 to D_F1, SW_A1 to SW_F1
Connections:
- net labels added: colG
Changed lines of the file:
@@
 Wire Wire Line
 	8250 2150 8250 2450
-Wire Wire Line
-	8950 2150 8950 2450
 Connection ~ 8850 5350
 Connection ~ 8850 4700
@@
 L foostan:SW_PUSH SW_A4
 U 1 1 5F6A8BBB
-P 9250 4400
-F 0 "SW_A4" H 9250 4655 50  0000 C CNN
-F 1 "SW_PUSH" H 9250 4564 50  0000 C CNN
-F 2 "local:CherryMX_Direct_Hotswap_Reversible" H 9250 4400 50  0001 C CNN
-F 3 "" H 9250 4400 50  0000 C CNN
-	1    9250 4400
-	1    0    0    -1
-$EndComp
-$Comp
-L foostan:SW_PUSH SW_A1
+P 5050 4400
+F 0 "SW_A4" H 5050 4655 50  0000 C CNN
+F 1 "SW_PUSH" H 5050 4564 50  0000 C CNN
+F 2 "local:CherryMX_Direct_Hotswap_Reversible" H 5050 4400 50  0001 C CNN
+F 3 "" H 5050 4400 50  0000 C CNN
+	1    5050 4400
+	1    0    0    -1
+$EndComp
+$Comp
+L foostan:SW_PUSH SW_F1
 U 1 1 5F6AA817
-P 9250 2450
-F 0 "SW_A1" H 9250 2705 50  0000 C CNN
-F 1 "SW_PUSH" H 9250 2614 50  0000 C CNN
-F 2 "local:CherryMX_Direct_Hotswap_Reversible" H 9250 2450 50  0001 C CNN
-F 3 "" H 9250 2450 50  0000 C CNN
-	1    9250 2450
+P 5750 2450
+F 0 "SW_F1" H 5750 2705 50  0000 C CNN
+F 1 "SW_PUSH" H 5750 2614 50  0000 C CNN
+F 2 "local:CherryMX_Direct_Hotswap_Reversible" H 5750 2450 50  0001 C CNN
+F 3 "" H 5750 2450 50  0000 C CNN
+	1    5750 2450
 	1    0    0    -1
 $EndComp
@@
 Wire Wire Line
 	8850 4050 9550 4050
-Connection ~ 9550 4050
-Wire Wire Line
-	8850 4700 9550 4700
-Connection ~ 9550 4700
-Connection ~ 9550 3400
-Connection ~ 9550 2750
 Wire Wire Line
 	8850 3400 9550 3400
-Wire Wire Line
-	9550 3400 9650 3400
 Text GLabel 8950 2150 0    50   Input ~ 0
 colA
 $Comp
-L Device:D D_A1
+L Device:D D_F1
 U 1 1 5F6AA821
-P 9550 2600
-F 0 "D_A1" V 9596 2680 50  0000 L CNN
-F 1 "D" V 9505 2680 50  0000 L CNN
-F 2 "foostan:D3_TH_SMD" H 9550 2600 50  0001 C CNN
-F 3 "~" H 9550 2600 50  0001 C CNN
-	1    9550 2600
+P 6050 2600
+F 0 "D_F1" V 6096 2680 50  0000 L CNN
+F 1 "D" V 6005 2680 50  0000 L CNN
+F 2 "foostan:D3_TH_SMD" H 6050 2600 50  0001 C CNN
+F 3 "~" H 6050 2600 50  0001 C CNN
+	1    6050 2600
 	0    -1   -1   0
 $EndComp
@@
 L Device:D D_A4
 U 1 1 5F6A8BC5
-P 9550 4550
-F 0 "D_A4" V 9596 4630 50  0000 L CNN
-F 1 "D" V 9505 4630 50  0000 L CNN
-F 2 "foostan:D3_TH_SMD" H 9550 4550 50  0001 C CNN
-F 3 "~" H 9550 4550 50  0001 C CNN
-	1    9550 4550
+P 5350 4550
+F 0 "D_A4" V 5396 4630 50  0000 L CNN
+F 1 "D" V 5305 4630 50  0000 L CNN
+F 2 "foostan:D3_TH_SMD" H 5350 4550 50  0001 C CNN
+F 3 "~" H 5350 4550 50  0001 C CNN
+	1    5350 4550
 	0    -1   -1   0
 $EndComp
@@
 Text GLabel 9650 4700 2    50   Input ~ 0
 row4
-Text GLabel 9650 4050 2    50   Input ~ 0
-row3
-Text GLabel 9650 3400 2    50   Input ~ 0
-row2
-Text GLabel 9650 2750 2    50   Input ~ 0
-row1
 Connection ~ 8250 2450
 Wire Wire Line
@@
 	8250 3750 8250 4400
 Connection ~ 8250 4400
-Connection ~ 8950 2450
-Wire Wire Line
-	8950 2450 8950 3100
 Connection ~ 8950 3100
 Wire Wire Line
 	8950 3100 8950 3750
 Connection ~ 8950 3750
-Wire Wire Line
-	8950 3750 8950 4400
 Wire Wire Line
 	8250 4400 8250 5050
@@
 Connection ~ 1550 6400
 Wire Wire Line
-	9550 4050 9650 4050
-Wire Wire Line
-	9550 4700 9650 4700
-Wire Wire Line
 	8150 5350 7450 5350
 Connection ~ 8150 5350
 Wire Wire Line
 	9550 5350 9650 5350
-Wire Wire Line
-	8950 5050 8950 4400
-Connection ~ 8950 4400
-Wire Wire Line
-	8850 2750 9550 2750
-Wire Wire Line
-	9550 2750 9650 2750
 $Comp
 L Device:D D_C3
@@
 Connection ~ 8150 3400
 Connection ~ 7450 3400
-Text GLabel 4250 3900 0    50   Input ~ 0
-B5
-Wire Wire Line
-	5450 2150 5450 2450
 Wire Wire Line
 	6150 2150 6150 2450
@@
 	5450 3100 5450 3750
 Connection ~ 6750 3400
-$Comp
-L local:joystick_s U3
-U 1 1 604A6B52
-P 4550 3900
-F 0 "U3" H 4778 3951 50  0000 L CNN
-F 1 "joystick_s" H 4778 3860 50  0000 L CNN
-F 2 "local:Joycon_Stick_Short" H 4550 3600 50  0001 C CNN
-F 3 "" H 4550 3600 50  0001 C CNN
-	1    4550 3900
-	1    0    0    -1
-$EndComp
-Text GLabel 4250 4100 0    50   Input ~ 0
-F4
-Text GLabel 4250 3800 0    50   Input ~ 0
-F5
-$Comp
-L power:VCC #PWR0108
-U 1 1 604BCAF5
-P 4250 3700
-F 0 "#PWR0108" H 4250 3550 50  0001 C CNN
-F 1 "VCC" H 4265 3873 50  0000 C CNN
-F 2 "" H 4250 3700 50  0001 C CNN
-F 3 "" H 4250 3700 50  0001 C CNN
-	1    4250 3700
-	1    0    0    -1
-$EndComp
-$Comp
-L power:GND #PWR0109
-U 1 1 604D24B1
-P 4000 4000
-F 0 "#PWR0109" H 4000 3750 50  0001 C CNN
-F 1 "GND" H 4005 3827 50  0000 C CNN
-F 2 "" H 4000 4000 50  0001 C CNN
-F 3 "" H 4000 4000 50  0001 C CNN
-	1    4000 4000
-	1    0    0    -1
-$EndComp
-Wire Wire Line
-	4250 4000 4000 4000
-$Comp
-L Device:Jumper JP_NOJS1
-U 1 1 604EEF7A
-P 3000 7000
-F 0 "JP_NOJS1" H 3000 6868 50  0000 C CNN
-F 1 "Jumper" H 3000 6777 50  0000 C CNN
-F 2 "Jumper:SolderJumper-2_P1.3mm_Open_RoundedPad1.0x1.5mm" H 3000 7000 50  0001 C CNN
-F 3 "~" H 3000 7000 50  0001 C CNN
-	1    3000 7000
-	1    0    0    -1
-$EndComp
-$Comp
-L power:GND #PWR0110
-U 1 1 604EF580
-P 3300 7000
-F 0 "#PWR0110" H 3300 6750 50  0001 C CNN
-F 1 "GND" H 3305 6827 50  0000 C CNN
-F 2 "" H 3300 7000 50  0001 C CNN
-F 3 "" H 3300 7000 50  0001 C CNN
-	1    3300 7000
-	1    0    0    -1
-$EndComp
-Text GLabel 2700 7000 0    50   Input ~ 0
-B5
-$Comp
-L foostan:SW_PUSH SW_F1
-U 1 1 605FBDAB
-P 5750 2450
-F 0 "SW_F1" H 5750 2705 50  0000 C CNN
-F 1 "SW_PUSH" H 5750 2614 50  0000 C CNN
-F 2 "local:CherryMX_Direct_Hotswap_Reversible" H 5750 2450 50  0001 C CNN
-F 3 "" H 5750 2450 50  0000 C CNN
-	1    5750 2450
-	1    0    0    -1
-$EndComp
+Wire Wire Line
+	5450 2150 5450 2450
+Wire Wire Line
+	2700 6600 3200 6600
+Text GLabel 3200 6600 2    50   Input ~ 0
+colG
+Text GLabel 2700 6600 0    50   Input ~ 0
+B4
+Connection ~ 9550 4050
+Wire Wire Line
+	9550 4050 9650 4050
+Text GLabel 9650 2750 2    50   Input ~ 0
+row1
+Connection ~ 9550 3400
+Wire Wire Line
+	9550 3400 9650 3400
+Text GLabel 4750 2150 0    50   Input ~ 0
+colG
+Connection ~ 4750 3100
+Wire Wire Line
+	4750 2150 4750 3100
+Wire Wire Line
+	4750 3100 4750 3750
+Connection ~ 6050 4050
+Connection ~ 6050 3400
+$Comp
+L foostan:SW_PUSH SW_G2
+U 1 1 60A7871B
+P 5050 3100
+F 0 "SW_G2" H 5050 3355 50  0000 C CNN
+F 1 "SW_PUSH" H 5050 3264 50  0000 C CNN
+F 2 "local:CherryMX_Direct_Hotswap_Reversible" H 5050 3100 50  0001 C CNN
+F 3 "" H 5050 3100 50  0000 C CNN
+	1    5050 3100
+	1    0    0    -1
+$EndComp
+$Comp
+L foostan:SW_PUSH SW_G3
+U 1 1 60A786E9
+P 5050 3750
+F 0 "SW_G3" H 5050 4005 50  0000 C CNN
+F 1 "SW_PUSH" H 5050 3914 50  0000 C CNN
+F 2 "local:CherryMX_Direct_Hotswap_Reversible" H 5050 3750 50  0001 C CNN
+F 3 "" H 5050 3750 50  0000 C CNN
+	1    5050 3750
+	1    0    0    -1
+$EndComp
+$Comp
+L Device:D D_G3
+U 1 1 60A786F3
+P 5350 3900
+F 0 "D_G3" V 5396 3980 50  0000 L CNN
+F 1 "D" V 5305 3980 50  0000 L CNN
+F 2 "foostan:D3_TH_SMD" H 5350 3900 50  0001 C CNN
+F 3 "~" H 5350 3900 50  0001 C CNN
+	1    5350 3900
+	0    -1   -1   0
+$EndComp
+$Comp
+L Device:D D_G2
+U 1 1 60A78711
+P 5350 3250
+F 0 "D_G2" V 5396 3330 50  0000 L CNN
+F 1 "D" V 5305 3330 50  0000 L CNN
+F 2 "foostan:D3_TH_SMD" H 5350 3250 50  0001 C CNN
+F 3 "~" H 5350 3250 50  0001 C CNN
+	1    5350 3250
+	0    -1   -1   0
+$EndComp
+Wire Wire Line
+	5350 4050 6050 4050
+Wire Wire Line
+	5350 3400 6050 3400
+Text GLabel 9650 3400 2    50   Input ~ 0
+row2
+Text GLabel 9650 4050 2    50   Input ~ 0
+row3
 Connection ~ 5450 2450
 Wire Wire Line
 	5450 2450 5450 3100
-$Comp
-L Device:D D_F1
-U 1 1 605FD473
-P 6050 2600
-F 0 "D_F1" V 6096 2680 50  0000 L CNN
-F 1 "D" V 6005 2680 50  0000 L CNN
-F 2 "foostan:D3_TH_SMD" H 6050 2600 50  0001 C CNN
-F 3 "~" H 6050 2600 50  0001 C CNN
-	1    6050 2600
-	0    -1   -1   0
-$EndComp
+Wire Wire Line
+	8950 2150 8950 3100
+Wire Wire Line
+	8850 2750 9650 2750
 Wire Wire Line
 	6750 2750 6050 2750
 Connection ~ 6750 2750
-$Comp
-L foostan:SW_PUSH SW_E5
-U 1 1 6060C4D7
-P 6450 5050
-F 0 "SW_E5" H 6450 5305 50  0000 C CNN
-F 1 "SW_PUSH" H 6450 5214 50  0000 C CNN
-F 2 "local:CherryMX_Direct_Hotswap_Reversible" H 6450 5050 50  0001 C CNN
-F 3 "" H 6450 5050 50  0000 C CNN
-	1    6450 5050
-	1    0    0    -1
-$EndComp
-Wire Wire Line
-	6150 4400 6150 5050
-Connection ~ 6150 4400
-$Comp
-L Device:D D_E5
-U 1 1 60616038
-P 6750 5200
-F 0 "D_E5" V 6796 5280 50  0000 L CNN
-F 1 "D" V 6705 5280 50  0000 L CNN
-F 2 "foostan:D3_TH_SMD" H 6750 5200 50  0001 C CNN
-F 3 "~" H 6750 5200 50  0001 C CNN
-	1    6750 5200
-	0    -1   -1   0
-$EndComp
-Wire Wire Line
-	7450 5350 6750 5350
-Connection ~ 7450 5350
+Wire Wire Line
+	8850 4700 9650 4700
+Wire Wire Line
+	8950 3750 8950 5050
+Wire Wire Line
+	4750 3750 4750 4400
+Connection ~ 4750 3750
+Wire Wire Line
+	6050 4700 5350 4700
+Connection ~ 6050 4700
 $EndSCHEMATC

Commit message: update sch
Parts:
- renumbered D_A4 to D_G4, SW_A4 to SW_G4
Changed lines of the file:
@@
 Title "Musashi50"
 Date ""
-Rev "8"
+Rev "B"
 Comp "HAMANO Tsukasa"
 Comment1 ""
@@
 $EndComp
 $Comp
-L foostan:SW_PUSH SW_A4
+L foostan:SW_PUSH SW_G4
 U 1 1 5F6A8BBB
 P 5050 4400
-F 0 "SW_A4" H 5050 4655 50  0000 C CNN
+F 0 "SW_G4" H 5050 4655 50  0000 C CNN
 F 1 "SW_PUSH" H 5050 4564 50  0000 C CNN
 F 2 "local:CherryMX_Direct_Hotswap_Reversible" H 5050 4400 50  0001 C CNN
@@
 $EndComp
 $Comp
-L Device:D D_A4
+L Device:D D_G4
 U 1 1 5F6A8BC5
 P 5350 4550
-F 0 "D_A4" V 5396 4630 50  0000 L CNN
+F 0 "D_G4" V 5396 4630 50  0000 L CNN
 F 1 "D" V 5305 4630 50  0000 L CNN
 F 2 "foostan:D3_TH_SMD" H 5350 4550 50  0001 C CNN

Commit message: add last key
Parts:
- added D_G1: D, foostan:D3_TH_SMD, symbol Device:D
- added SW_G1: SW_PUSH, local:CherryMX_Direct_Hotswap_Reversible, symbol foostan:SW_PUSH
Connections:
- wire segments 85 -> 87
Changed lines of the file:
@@
 Connection ~ 4750 3100
 Wire Wire Line
-	4750 2150 4750 3100
+	4750 2150 4750 2450
 Wire Wire Line
 	4750 3100 4750 3750
@@
 	6050 4700 5350 4700
 Connection ~ 6050 4700
+$Comp
+L foostan:SW_PUSH SW_G1
+U 1 1 60DF9883
+P 5050 2450
+F 0 "SW_G1" H 5050 2705 50  0000 C CNN
+F 1 "SW_PUSH" H 5050 2614 50  0000 C CNN
+F 2 "local:CherryMX_Direct_Hotswap_Reversible" H 5050 2450 50  0001 C CNN
+F 3 "" H 5050 2450 50  0000 C CNN
+	1    5050 2450
+	1    0    0    -1
+$EndComp
+Connection ~ 4750 2450
+Wire Wire Line
+	4750 2450 4750 3100
+$Comp
+L Device:D D_G1
+U 1 1 60DFA810
+P 5350 2600
+F 0 "D_G1" V 5396 2680 50  0000 L CNN
+F 1 "D" V 5305 2680 50  0000 L CNN
+F 2 "foostan:D3_TH_SMD" H 5350 2600 50  0001 C CNN
+F 3 "~" H 5350 2600 50  0001 C CNN
+	1    5350 2600
+	0    -1   -1   0
+$EndComp
+Wire Wire Line
+	6050 2750 5350 2750
+Connection ~ 6050 2750
 $EndSCHEMATC

Commit message: add revC sch
Parts:
- added OL1: OLED, Connector_PinSocket_2.54mm:PinSocket_1x04_P2.54mm_Vertical, symbol foostan:OLED
- JP_LEFT1: value Jumper -> JP_LEFT
- JP_RIGHT1: value Jumper -> JP_RIGHT
Connections:
- wire segments 87 -> 92
Changed lines of the file:
@@
 Text GLabel 1500 2900 0    50   Input ~ 0
 B3
-Text GLabel 2700 5400 0    50   Input ~ 0
+Text GLabel 2450 5300 0    50   Input ~ 0
 D1
-Text GLabel 3200 5400 2    50   Input ~ 0
+Text GLabel 1300 5300 0    50   Input ~ 0
 colA
 Wire Wire Line
-	2700 5400 3200 5400
-Text GLabel 2700 5600 0    50   Input ~ 0
+	2450 5300 3650 5300
+Text GLabel 2450 5500 0    50   Input ~ 0
 D0
-Text GLabel 3200 5600 2    50   Input ~ 0
+Text GLabel 1300 5500 0    50   Input ~ 0
 colB
 Wire Wire Line
-	2700 5600 3200 5600
+	2450 5500 3800 5500
 Text GLabel 1500 3000 0    50   Input ~ 0
 B2
@@
 	1    0    0    -1
 $EndComp
-Text GLabel 2700 5800 0    50   Input ~ 0
+Text GLabel 2450 5700 0    50   Input ~ 0
 D4
-Text GLabel 3200 5800 2    50   Input ~ 0
+Text GLabel 1300 5700 0    50   Input ~ 0
 colC
 Wire Wire Line
-	2700 5800 3200 5800
+	2450 5700 2950 5700
 Text GLabel 2900 2600 2    50   Input ~ 0
 D4
@@
 	0    -1   -1   0
 $EndComp
-Text GLabel 2700 6000 0    50   Input ~ 0
+Text GLabel 2450 5900 0    50   Input ~ 0
 C6
-Text GLabel 3200 6000 2    50   Input ~ 0
+Text GLabel 1300 5900 0    50   Input ~ 0
 colD
 Wire Wire Line
-	2700 6000 3200 6000
-Text GLabel 2700 6200 0    50   Input ~ 0
+	2450 5900 2950 5900
+Text GLabel 2450 6100 0    50   Input ~ 0
 D7
-Text GLabel 3200 6200 2    50   Input ~ 0
+Text GLabel 1300 6100 0    50   Input ~ 0
 colE
 Wire Wire Line
-	2700 6200 3200 6200
-Text GLabel 2700 6400 0    50   Input ~ 0
+	2450 6100 2950 6100
+Text GLabel 2450 6300 0    50   Input ~ 0
 E6
-Text GLabel 3200 6400 2    50   Input ~ 0
+Text GLabel 1300 6300 0    50   Input ~ 0
 colF
 Wire Wire Line
-	2700 6400 3200 6400
+	2450 6300 2950 6300
 Text GLabel 2900 2700 2    50   Input ~ 0
 C6
@@
 D3
 Wire Wire Line
-	2050 6200 1550 6200
-Text GLabel 1550 6200 0    50   Input ~ 0
-row5
-Text GLabel 2050 6200 2    50   Input ~ 0
+	1800 6500 1300 6500
+Text GLabel 1800 6500 2    50   Input ~ 0
 B2
 Wire Wire Line
-	2050 6000 1550 6000
-Text GLabel 1550 6000 0    50   Input ~ 0
-row4
-Text GLabel 2050 6000 2    50   Input ~ 0
+	1800 6300 1300 6300
+Text GLabel 1800 6300 2    50   Input ~ 0
 B3
 Wire Wire Line
-	2050 5800 1550 5800
-Text GLabel 1550 5800 0    50   Input ~ 0
-row3
-Text GLabel 2050 5800 2    50   Input ~ 0
+	1800 6100 1300 6100
+Text GLabel 1800 6100 2    50   Input ~ 0
 B1
 Wire Wire Line
-	2050 5600 1550 5600
-Text GLabel 1550 5600 0    50   Input ~ 0
-row2
-Wire Wire Line
-	2050 5400 1550 5400
-Text GLabel 1550 5400 0    50   Input ~ 0
-row1
-Text GLabel 2700 5200 0    50   Input ~ 0
+	1800 5900 1300 5900
+Wire Wire Line
+	1800 5700 1300 5700
+Text GLabel 2450 5100 0    50   Input ~ 0
 D2
-Text GLabel 3200 5200 2    50   Input ~ 0
+Text GLabel 2950 5100 2    50   Input ~ 0
 data
 Wire Wire Line
-	2700 5200 3200 5200
-Wire Wire Line
-	2050 6400 1550 6400
-Text GLabel 2050 6400 2    50   Input ~ 0
+	2450 5100 2950 5100
+Wire Wire Line
+	1800 6700 1300 6700
+Text GLabel 1800 6700 2    50   Input ~ 0
 B6
 $Comp
 L Device:Jumper JP_LEFT1
 U 1 1 5F738159
-P 1250 6400
-F 0 "JP_LEFT1" H 1250 6268 50  0000 C CNN
-F 1 "Jumper" H 1250 6177 50  0000 C CNN
-F 2 "Jumper:SolderJumper-2_P1.3mm_Open_RoundedPad1.0x1.5mm" H 1250 6400 50  0001 C CNN
-F 3 "~" H 1250 6400 50  0001 C CNN
-	1    1250 6400
+P 1000 6700
+F 0 "JP_LEFT1" H 1000 6568 50  0001 C CNN
+F 1 "JP_LEFT" H 1000 6477 50  0000 C CNN
+F 2 "Jumper:SolderJumper-2_P1.3mm_Open_RoundedPad1.0x1.5mm" H 1000 6700 50  0001 C CNN
+F 3 "~" H 1000 6700 50  0001 C CNN
+	1    1000 6700
 	1    0    0    -1
 $EndComp
@@
 	3050 3925 3050 4125
 NoConn ~ 2850 3825
-Text GLabel 2050 5400 2    50   Input ~ 0
-F6
-Text GLabel 2050 5600 2    50   Input ~ 0
+Text GLabel 1800 5900 2    50   Input ~ 0
 F7
 Text GLabel 1500 2400 0    50   Input ~ 0
@@
 L Device:Jumper JP_RIGHT1
 U 1 1 5F795429
-P 1250 6850
-F 0 "JP_RIGHT1" H 1250 6718 50  0000 C CNN
-F 1 "Jumper" H 1250 6627 50  0000 C CNN
-F 2 "Jumper:SolderJumper-2_P1.3mm_Open_RoundedPad1.0x1.5mm" H 1250 6850 50  0001 C CNN
-F 3 "~" H 1250 6850 50  0001 C CNN
-	1    1250 6850
+P 1000 7150
+F 0 "JP_RIGHT1" H 1000 7018 50  0001 C CNN
+F 1 "JP_RIGHT" H 1000 6927 50  0000 C CNN
+F 2 "Jumper:SolderJumper-2_P1.3mm_Open_RoundedPad1.0x1.5mm" H 1000 7150 50  0001 C CNN
+F 3 "~" H 1000 7150 50  0001 C CNN
+	1    1000 7150
 	1    0    0    -1
 $EndComp
@@
 L power:GND #PWR05
 U 1 1 5F79542F
-P 950 6850
-F 0 "#PWR05" H 950 6600 50  0001 C CNN
-F 1 "GND" H 955 6677 50  0000 C CNN
-F 2 "" H 950 6850 50  0001 C CNN
-F 3 "" H 950 6850 50  0001 C CNN
-	1    950  6850
+P 700 7150
+F 0 "#PWR05" H 700 6900 50  0001 C CNN
+F 1 "GND" H 705 6977 50  0000 C CNN
+F 2 "" H 700 7150 50  0001 C CNN
+F 3 "" H 700 7150 50  0001 C CNN
+	1    700  7150
 	1    0    0    -1
 $EndComp
@@
 L power:VCC #PWR02
 U 1 1 5F7A2499
-P 950 6400
-F 0 "#PWR02" H 950 6250 50  0001 C CNN
-F 1 "VCC" H 965 6573 50  0000 C CNN
-F 2 "" H 950 6400 50  0001 C CNN
-F 3 "" H 950 6400 50  0001 C CNN
-	1    950  6400
-	1    0    0    -1
-$EndComp
-Wire Wire Line
-	1550 6400 1550 6850
-Connection ~ 1550 6400
+P 700 6700
+F 0 "#PWR02" H 700 6550 50  0001 C CNN
+F 1 "VCC" H 715 6873 50  0000 C CNN
+F 2 "" H 700 6700 50  0001 C CNN
+F 3 "" H 700 6700 50  0001 C CNN
+	1    700  6700
+	1    0    0    -1
+$EndComp
+Wire Wire Line
+	1300 6700 1300 7150
+Connection ~ 1300 6700
 Wire Wire Line
 	8150 5350 7450 5350
@@
 	5450 2150 5450 2450
 Wire Wire Line
-	2700 6600 3200 6600
-Text GLabel 3200 6600 2    50   Input ~ 0
+	2450 6500 2950 6500
+Text GLabel 1300 6500 0    50   Input ~ 0
 colG
-Text GLabel 2700 6600 0    50   Input ~ 0
+Text GLabel 2450 6500 0    50   Input ~ 0
 B4
 Connection ~ 9550 4050
@@
 	6050 2750 5350 2750
 Connection ~ 6050 2750
+$Comp
+L foostan:OLED OL1
+U 1 1 60E710A5
+P 3900 4550
+F 0 "OL1" H 4528 4619 51  0000 L CNN
+F 1 "OLED" H 4528 4529 47  0000 L CNN
+F 2 "Connector_PinSocket_2.54mm:PinSocket_1x04_P2.54mm_Vertical" H 3900 4650 60  0001 C CNN
+F 3 "" H 3900 4650 60  0001 C CNN
+	1    3900 4550
+	0    -1   -1   0
+$EndComp
+Text GLabel 2950 5700 2    50   Input ~ 0
+row1
+Text GLabel 2950 5900 2    50   Input ~ 0
+row2
+Text GLabel 2950 6100 2    50   Input ~ 0
+row3
+Text GLabel 2950 6300 2    50   Input ~ 0
+row4
+Text GLabel 2950 6500 2    50   Input ~ 0
+row5
+Wire Wire Line
+	1800 5500 1300 5500
+Wire Wire Line
+	1800 5300 1300 5300
+Text GLabel 1800 5300 2    50   Input ~ 0
+F4
+Text GLabel 1800 5500 2    50   Input ~ 0
+F5
+Text GLabel 1800 5700 2    50   Input ~ 0
+F6
+Wire Wire Line
+	3800 5500 3800 5300
+$Comp
+L power:VCC #PWR03
+U 1 1 60F35351
+P 3950 5500
+F 0 "#PWR03" H 3950 5350 50  0001 C CNN
+F 1 "VCC" H 3965 5673 50  0000 C CNN
+F 2 "" H 3950 5500 50  0001 C CNN
+F 3 "" H 3950 5500 50  0001 C CNN
+	1    3950 5500
+	1    0    0    1
+$EndComp
+$Comp
+L power:GND #PWR04
+U 1 1 60F37C22
+P 4100 5500
+F 0 "#PWR04" H 4100 5250 50  0001 C CNN
+F 1 "GND" H 4105 5327 50  0000 C CNN
+F 2 "" H 4100 5500 50  0001 C CNN
+F 3 "" H 4100 5500 50  0001 C CNN
+	1    4100 5500
+	1    0    0    -1
+$EndComp
+Wire Wire Line
+	3950 5300 3950 5500
+Wire Wire Line
+	4100 5300 4100 5500
 $EndSCHEMATC
