File: pcb/musashi60.sch (KiCad schematic (older format))
At the start: 66 parts, among them J1 MJ-4PP-9, U1 ProMicro_r

Commit message: update revD scheme
Parts:
- JP_LEFT1, JP_RIGHT1: footprint Jumper:SolderJumper-2_P1.3mm_Open_RoundedPad1.0x1.5mm -> local:SolderJumper
- OL1: footprint Connector_PinSocket_2.54mm:PinSocket_1x04_P2.54mm_Vertical -> local:OLED_Reversible
- SW_RST1: footprint foostan:ResetSW -> local:ResetSW
- U1: footprint foostan:ProMicro_v2 -> local:ProMicro
Connections:
- no-connect marks 2 -> 4
Changed lines of the file:
@@
 F 0 "U1" H 2200 3687 60  0000 C CNN
 F 1 "ProMicro_r" H 2200 3581 60  0000 C CNN
-F 2 "foostan:ProMicro_v2" H 2300 1650 60  0001 C CNN
+F 2 "local:ProMicro" H 2300 1650 60  0001 C CNN
 F 3 "" H 2300 1650 60  0000 C CNN
 	1    2150 2700
@@
 F 0 "SW_RST1" H 1450 4205 50  0000 C CNN
 F 1 "SW_PUSH" H 1450 4114 50  0000 C CNN
-F 2 "foostan:ResetSW" H 1450 3950 50  0001 C CNN
+F 2 "local:ResetSW" H 1450 3950 50  0001 C CNN
 F 3 "" H 1450 3950 50  0000 C CNN
 	1    1450 3950
@@
 F 0 "JP_LEFT1" H 1000 6568 50  0001 C CNN
 F 1 "JP_LEFT" H 1000 6477 50  0000 C CNN
-F 2 "Jumper:SolderJumper-2_P1.3mm_Open_RoundedPad1.0x1.5mm" H 1000 6700 50  0001 C CNN
+F 2 "local:SolderJumper" H 1000 6700 50  0001 C CNN
 F 3 "~" H 1000 6700 50  0001 C CNN
 	1    1000 6700
@@
 F 0 "JP_RIGHT1" H 1000 7018 50  0001 C CNN
 F 1 "JP_RIGHT" H 1000 6927 50  0000 C CNN
-F 2 "Jumper:SolderJumper-2_P1.3mm_Open_RoundedPad1.0x1.5mm" H 1000 7150 50  0001 C CNN
+F 2 "local:SolderJumper" H 1000 7150 50  0001 C CNN
 F 3 "~" H 1000 7150 50  0001 C CNN
 	1    1000 7150
@@
 F 0 "OL1" H 4528 4619 51  0000 L CNN
 F 1 "OLED" H 4528 4529 47  0000 L CNN
-F 2 "Connector_PinSocket_2.54mm:PinSocket_1x04_P2.54mm_Vertical" H 3900 4650 60  0001 C CNN
+F 2 "local:OLED_Reversible" H 3900 4650 60  0001 C CNN
 F 3 "" H 3900 4650 60  0001 C CNN
 	1    3900 4550
@@
 Wire Wire Line
 	4100 5300 4100 5500
+Text GLabel 2450 6700 0    50   Input ~ 0
+B5
+NoConn ~ 2450 6700
+Text GLabel 2450 4900 0    50   Input ~ 0
+D3
+NoConn ~ 2450 4900
 $EndSCHEMATC

Commit message: update scheme for revD
Parts:
- added U2: OLED_Reversible_Jumper, local:OLED_Reversible_Jumper, symbol local:OLED_Reversible_Jumper
- D_A2, D_A3, D_A5, D_B1, D_B2, D_B3, D_B4, D_B5, D_C1, D_C2, D_C3, D_C4, D_C5, D_D1, D_D2, D_D3, D_D4, D_D5, D_E1, D_E2, D_E3, D_E4, D_F1, D_F2, D_F3, D_F4, D_G1, D_G2, D_G3, D_G4: footprint foostan:D3_TH_SMD -> local:D_TH
Connections:
- wire segments 92 -> 98
Changed lines of the file:
@@
 colA
 Wire Wire Line
-	2450 5300 3650 5300
-Text GLabel 2450 5500 0    50   Input ~ 0
-D0
+	2450 5300 3500 5300
 Text GLabel 1300 5500 0    50   Input ~ 0
 colB
-Wire Wire Line
-	2450 5500 3800 5500
 Text GLabel 1500 3000 0    50   Input ~ 0
 B2
@@
 	1    0    0    -1
 $EndComp
-Text GLabel 2450 5700 0    50   Input ~ 0
-D4
 Text GLabel 1300 5700 0    50   Input ~ 0
 colC
-Wire Wire Line
-	2450 5700 2950 5700
 Text GLabel 2900 2600 2    50   Input ~ 0
 D4
@@
 F 0 "D_B3" V 8896 3980 50  0000 L CNN
 F 1 "D" V 8805 3980 50  0000 L CNN
-F 2 "foostan:D3_TH_SMD" H 8850 3900 50  0001 C CNN
+F 2 "local:D_TH" H 8850 3900 50  0001 C CNN
 F 3 "~" H 8850 3900 50  0001 C CNN
 	1    8850 3900
@@
 F 0 "D_B2" V 8896 3330 50  0000 L CNN
 F 1 "D" V 8805 3330 50  0000 L CNN
-F 2 "foostan:D3_TH_SMD" H 8850 3250 50  0001 C CNN
+F 2 "local:D_TH" H 8850 3250 50  0001 C CNN
 F 3 "~" H 8850 3250 50  0001 C CNN
 	1    8850 3250
@@
 F 0 "D_B1" V 8896 2680 50  0000 L CNN
 F 1 "D" V 8805 2680 50  0000 L CNN
-F 2 "foostan:D3_TH_SMD" H 8850 2600 50  0001 C CNN
+F 2 "local:D_TH" H 8850 2600 50  0001 C CNN
 F 3 "~" H 8850 2600 50  0001 C CNN
 	1    8850 2600
@@
 F 0 "D_B4" V 8896 4630 50  0000 L CNN
 F 1 "D" V 8805 4630 50  0000 L CNN
-F 2 "foostan:D3_TH_SMD" H 8850 4550 50  0001 C CNN
+F 2 "local:D_TH" H 8850 4550 50  0001 C CNN
 F 3 "~" H 8850 4550 50  0001 C CNN
 	1    8850 4550
@@
 F 0 "D_C5" V 8196 5280 50  0000 L CNN
 F 1 "D" V 8105 5280 50  0000 L CNN
-F 2 "foostan:D3_TH_SMD" H 8150 5200 50  0001 C CNN
+F 2 "local:D_TH" H 8150 5200 50  0001 C CNN
 F 3 "~" H 8150 5200 50  0001 C CNN
 	1    8150 5200
@@
 F 0 "D_A3" V 9596 3980 50  0000 L CNN
 F 1 "D" V 9505 3980 50  0000 L CNN
-F 2 "foostan:D3_TH_SMD" H 9550 3900 50  0001 C CNN
+F 2 "local:D_TH" H 9550 3900 50  0001 C CNN
 F 3 "~" H 9550 3900 50  0001 C CNN
 	1    9550 3900
@@
 F 0 "D_A2" V 9596 3330 50  0000 L CNN
 F 1 "D" V 9505 3330 50  0000 L CNN
-F 2 "foostan:D3_TH_SMD" H 9550 3250 50  0001 C CNN
+F 2 "local:D_TH" H 9550 3250 50  0001 C CNN
 F 3 "~" H 9550 3250 50  0001 C CNN
 	1    9550 3250
@@
 F 0 "D_F1" V 6096 2680 50  0000 L CNN
 F 1 "D" V 6005 2680 50  0000 L CNN
-F 2 "foostan:D3_TH_SMD" H 6050 2600 50  0001 C CNN
+F 2 "local:D_TH" H 6050 2600 50  0001 C CNN
 F 3 "~" H 6050 2600 50  0001 C CNN
 	1    6050 2600
@@
 F 0 "D_G4" V 5396 4630 50  0000 L CNN
 F 1 "D" V 5305 4630 50  0000 L CNN
-F 2 "foostan:D3_TH_SMD" H 5350 4550 50  0001 C CNN
+F 2 "local:D_TH" H 5350 4550 50  0001 C CNN
 F 3 "~" H 5350 4550 50  0001 C CNN
 	1    5350 4550
@@
 F 0 "D_B5" V 8896 5280 50  0000 L CNN
 F 1 "D" V 8805 5280 50  0000 L CNN
-F 2 "foostan:D3_TH_SMD" H 8850 5200 50  0001 C CNN
+F 2 "local:D_TH" H 8850 5200 50  0001 C CNN
 F 3 "~" H 8850 5200 50  0001 C CNN
 	1    8850 5200
@@
 F 0 "D_A5" V 9596 5279 50  0000 L CNN
 F 1 "D" V 9505 5279 50  0000 L CNN
-F 2 "foostan:D3_TH_SMD" H 9550 5200 50  0001 C CNN
+F 2 "local:D_TH" H 9550 5200 50  0001 C CNN
 F 3 "~" H 9550 5200 50  0001 C CNN
 	1    9550 5200
@@
 F 0 "D_D3" V 7496 3980 50  0000 L CNN
 F 1 "D" V 7405 3980 50  0000 L CNN
-F 2 "foostan:D3_TH_SMD" H 7450 3900 50  0001 C CNN
+F 2 "local:D_TH" H 7450 3900 50  0001 C CNN
 F 3 "~" H 7450 3900 50  0001 C CNN
 	1    7450 3900
@@
 F 0 "D_D2" V 7496 3330 50  0000 L CNN
 F 1 "D" V 7405 3330 50  0000 L CNN
-F 2 "foostan:D3_TH_SMD" H 7450 3250 50  0001 C CNN
+F 2 "local:D_TH" H 7450 3250 50  0001 C CNN
 F 3 "~" H 7450 3250 50  0001 C CNN
 	1    7450 3250
@@
 F 0 "D_D1" V 7496 2680 50  0000 L CNN
 F 1 "D" V 7405 2680 50  0000 L CNN
-F 2 "foostan:D3_TH_SMD" H 7450 2600 50  0001 C CNN
+F 2 "local:D_TH" H 7450 2600 50  0001 C CNN
 F 3 "~" H 7450 2600 50  0001 C CNN
 	1    7450 2600
@@
 F 0 "D_D4" V 7496 4630 50  0000 L CNN
 F 1 "D" V 7405 4630 50  0000 L CNN
-F 2 "foostan:D3_TH_SMD" H 7450 4550 50  0001 C CNN
+F 2 "local:D_TH" H 7450 4550 50  0001 C CNN
 F 3 "~" H 7450 4550 50  0001 C CNN
 	1    7450 4550
@@
 F 0 "D_D5" V 7496 5280 50  0000 L CNN
 F 1 "D" V 7405 5280 50  0000 L CNN
-F 2 "foostan:D3_TH_SMD" H 7450 5200 50  0001 C CNN
+F 2 "local:D_TH" H 7450 5200 50  0001 C CNN
 F 3 "~" H 7450 5200 50  0001 C CNN
 	1    7450 5200
@@
 F 0 "D_E3" V 6796 3980 50  0000 L CNN
 F 1 "D" V 6705 3980 50  0000 L CNN
-F 2 "foostan:D3_TH_SMD" H 6750 3900 50  0001 C CNN
+F 2 "local:D_TH" H 6750 3900 50  0001 C CNN
 F 3 "~" H 6750 3900 50  0001 C CNN
 	1    6750 3900
@@
 F 0 "D_E2" V 6796 3330 50  0000 L CNN
 F 1 "D" V 6705 3330 50  0000 L CNN
-F 2 "foostan:D3_TH_SMD" H 6750 3250 50  0001 C CNN
+F 2 "local:D_TH" H 6750 3250 50  0001 C CNN
 F 3 "~" H 6750 3250 50  0001 C CNN
 	1    6750 3250
@@
 F 0 "D_E1" V 6796 2680 50  0000 L CNN
 F 1 "D" V 6705 2680 50  0000 L CNN
-F 2 "foostan:D3_TH_SMD" H 6750 2600 50  0001 C CNN
+F 2 "local:D_TH" H 6750 2600 50  0001 C CNN
 F 3 "~" H 6750 2600 50  0001 C CNN
 	1    6750 2600
@@
 F 0 "D_E4" V 6796 4630 50  0000 L CNN
 F 1 "D" V 6705 4630 50  0000 L CNN
-F 2 "foostan:D3_TH_SMD" H 6750 4550 50  0001 C CNN
+F 2 "local:D_TH" H 6750 4550 50  0001 C CNN
 F 3 "~" H 6750 4550 50  0001 C CNN
 	1    6750 4550
@@
 F 0 "D_F3" V 6096 3980 50  0000 L CNN
 F 1 "D" V 6005 3980 50  0000 L CNN
-F 2 "foostan:D3_TH_SMD" H 6050 3900 50  0001 C CNN
+F 2 "local:D_TH" H 6050 3900 50  0001 C CNN
 F 3 "~" H 6050 3900 50  0001 C CNN
 	1    6050 3900
@@
 F 0 "D_F4" V 6096 4630 50  0000 L CNN
 F 1 "D" V 6005 4630 50  0000 L CNN
-F 2 "foostan:D3_TH_SMD" H 6050 4550 50  0001 C CNN
+F 2 "local:D_TH" H 6050 4550 50  0001 C CNN
 F 3 "~" H 6050 4550 50  0001 C CNN
 	1    6050 4550
@@
 F 0 "D_C1" V 8196 2680 50  0000 L CNN
 F 1 "D" V 8105 2680 50  0000 L CNN
-F 2 "foostan:D3_TH_SMD" H 8150 2600 50  0001 C CNN
+F 2 "local:D_TH" H 8150 2600 50  0001 C CNN
 F 3 "~" H 8150 2600 50  0001 C CNN
 	1    8150 2600
@@
 F 0 "D_F2" V 6096 3330 50  0000 L CNN
 F 1 "D" V 6005 3330 50  0000 L CNN
-F 2 "foostan:D3_TH_SMD" H 6050 3250 50  0001 C CNN
+F 2 "local:D_TH" H 6050 3250 50  0001 C CNN
 F 3 "~" H 6050 3250 50  0001 C CNN
 	1    6050 3250
@@
 F 0 "D_C2" V 8196 3330 50  0000 L CNN
 F 1 "D" V 8105 3330 50  0000 L CNN
-F 2 "foostan:D3_TH_SMD" H 8150 3250 50  0001 C CNN
+F 2 "local:D_TH" H 8150 3250 50  0001 C CNN
 F 3 "~" H 8150 3250 50  0001 C CNN
 	1    8150 3250
@@
 F 0 "D_C3" V 8196 3980 50  0000 L CNN
 F 1 "D" V 8105 3980 50  0000 L CNN
-F 2 "foostan:D3_TH_SMD" H 8150 3900 50  0001 C CNN
+F 2 "local:D_TH" H 8150 3900 50  0001 C CNN
 F 3 "~" H 8150 3900 50  0001 C CNN
 	1    8150 3900
@@
 F 0 "D_C4" V 8196 4630 50  0000 L CNN
 F 1 "D" V 8105 4630 50  0000 L CNN
-F 2 "foostan:D3_TH_SMD" H 8150 4550 50  0001 C CNN
+F 2 "local:D_TH" H 8150 4550 50  0001 C CNN
 F 3 "~" H 8150 4550 50  0001 C CNN
 	1    8150 4550
@@
 F 0 "D_G3" V 5396 3980 50  0000 L CNN
 F 1 "D" V 5305 3980 50  0000 L CNN
-F 2 "foostan:D3_TH_SMD" H 5350 3900 50  0001 C CNN
+F 2 "local:D_TH" H 5350 3900 50  0001 C CNN
 F 3 "~" H 5350 3900 50  0001 C CNN
 	1    5350 3900
@@
 F 0 "D_G2" V 5396 3330 50  0000 L CNN
 F 1 "D" V 5305 3330 50  0000 L CNN
-F 2 "foostan:D3_TH_SMD" H 5350 3250 50  0001 C CNN
+F 2 "local:D_TH" H 5350 3250 50  0001 C CNN
 F 3 "~" H 5350 3250 50  0001 C CNN
 	1    5350 3250
@@
 F 0 "D_G1" V 5396 2680 50  0000 L CNN
 F 1 "D" V 5305 2680 50  0000 L CNN
-F 2 "foostan:D3_TH_SMD" H 5350 2600 50  0001 C CNN
+F 2 "local:D_TH" H 5350 2600 50  0001 C CNN
 F 3 "~" H 5350 2600 50  0001 C CNN
 	1    5350 2600
@@
 L foostan:OLED OL1
 U 1 1 60E710A5
-P 3900 4550
-F 0 "OL1" H 4528 4619 51  0000 L CNN
-F 1 "OLED" H 4528 4529 47  0000 L CNN
-F 2 "local:OLED_Reversible" H 3900 4650 60  0001 C CNN
-F 3 "" H 3900 4650 60  0001 C CNN
-	1    3900 4550
-	0    -1   -1   0
-$EndComp
-Text GLabel 2950 5700 2    50   Input ~ 0
-row1
+P 4400 6650
+F 0 "OL1" H 5028 6719 51  0000 L CNN
+F 1 "OLED" H 5028 6629 47  0000 L CNN
+F 2 "local:OLED_Reversible" H 4400 6750 60  0001 C CNN
+F 3 "" H 4400 6750 60  0001 C CNN
+	1    4400 6650
+	0    1    1    0
+$EndComp
 Text GLabel 2950 5900 2    50   Input ~ 0
 row2
@@
 Text GLabel 1800 5700 2    50   Input ~ 0
 F6
-Wire Wire Line
-	3800 5500 3800 5300
 $Comp
 L power:VCC #PWR03
 U 1 1 60F35351
-P 3950 5500
-F 0 "#PWR03" H 3950 5350 50  0001 C CNN
-F 1 "VCC" H 3965 5673 50  0000 C CNN
-F 2 "" H 3950 5500 50  0001 C CNN
-F 3 "" H 3950 5500 50  0001 C CNN
-	1    3950 5500
+P 3300 6100
+F 0 "#PWR03" H 3300 5950 50  0001 C CNN
+F 1 "VCC" H 3315 6273 50  0000 C CNN
+F 2 "" H 3300 6100 50  0001 C CNN
+F 3 "" H 3300 6100 50  0001 C CNN
+	1    3300 6100
 	1    0    0    1
 $EndComp
@@
 L power:GND #PWR04
 U 1 1 60F37C22
-P 4100 5500
-F 0 "#PWR04" H 4100 5250 50  0001 C CNN
-F 1 "GND" H 4105 5327 50  0000 C CNN
-F 2 "" H 4100 5500 50  0001 C CNN
-F 3 "" H 4100 5500 50  0001 C CNN
-	1    4100 5500
-	1    0    0    -1
-$EndComp
-Wire Wire Line
-	3950 5300 3950 5500
-Wire Wire Line
-	4100 5300 4100 5500
+P 3500 6100
+F 0 "#PWR04" H 3500 5850 50  0001 C CNN
+F 1 "GND" H 3505 5927 50  0000 C CNN
+F 2 "" H 3500 6100 50  0001 C CNN
+F 3 "" H 3500 6100 50  0001 C CNN
+	1    3500 6100
+	1    0    0    -1
+$EndComp
+Wire Wire Line
+	3300 5700 3300 6100
+Wire Wire Line
+	3500 5900 3500 6100
 Text GLabel 2450 6700 0    50   Input ~ 0
 B5
@@
 D3
 NoConn ~ 2450 4900
+Text GLabel 2950 5700 2    50   Input ~ 0
+row1
+Wire Wire Line
+	2450 5700 2950 5700
+Text GLabel 2450 5700 0    50   Input ~ 0
+D4
+Wire Wire Line
+	2450 5500 3500 5500
+Text GLabel 2450 5500 0    50   Input ~ 0
+D0
+$Comp
+L local:OLED_Reversible_Jumper U2
+U 1 1 610EF83F
+P 3850 5100
+F 0 "U2" H 3850 5165 50  0000 C CNN
+F 1 "OLED_Reversible_Jumper" H 3850 5074 50  0000 C CNN
+F 2 "local:OLED_Reversible_Jumper" H 3850 5100 50  0001 C CNN
+F 3 "" H 3850 5100 50  0001 C CNN
+	1    3850 5100
+	1    0    0    -1
+$EndComp
+Wire Wire Line
+	3300 5700 3500 5700
+Wire Wire Line
+	4200 5700 4350 5700
+Wire Wire Line
+	4350 5700 4350 5900
+Wire Wire Line
+	4200 5500 4500 5500
+Wire Wire Line
+	4500 5500 4500 5900
+Wire Wire Line
+	4200 5300 4650 5300
+Wire Wire Line
+	4650 5300 4650 5900
 $EndSCHEMATC
