File: pcb/musashi50.sch (KiCad schematic (older format))
At the start: 66 parts, among them J1 MJ-4PP-9, U1 ProMicro_r, U2 joystick

Commit message: update rev9
Parts:
- removed B5: MountingHole_Pad, foostan:1pin_conn, symbol Mechanical:MountingHole_Pad
- added JP_NOJS1: Jumper, Jumper:SolderJumper-2_P1.3mm_Open_RoundedPad1.0x1.5mm, symbol Device:Jumper
- added U3: joystick_s, local:Joycon_Stick, symbol local:joystick_s
Changed lines of the file:
@@
 Title "Musashi50"
 Date ""
-Rev "9"
+Rev "8"
 Comp "HAMANO Tsukasa"
 Comment1 ""
@@
 L foostan:MJ-4PP-9 J1
 U 1 1 5F7A2FFF
-P 3400 3800
-F 0 "J1" H 3431 4076 50  0000 C CNN
-F 1 "MJ-4PP-9" H 3431 3985 50  0000 C CNN
-F 2 "foostan:MJ-4PP-9" H 3675 3975 50  0001 C CNN
-F 3 "~" H 3675 3975 50  0001 C CNN
-	1    3400 3800
+P 2650 3900
+F 0 "J1" H 2681 4176 50  0000 C CNN
+F 1 "MJ-4PP-9" H 2681 4085 50  0000 C CNN
+F 2 "foostan:MJ-4PP-9" H 2925 4075 50  0001 C CNN
+F 3 "~" H 2925 4075 50  0001 C CNN
+	1    2650 3900
 	1    0    0    -1
 $EndComp
@@
 L power:GND #PWR0106
 U 1 1 5F7AB1C4
-P 3800 4025
-F 0 "#PWR0106" H 3800 3775 50  0001 C CNN
-F 1 "GND" H 3805 3852 50  0000 C CNN
-F 2 "" H 3800 4025 50  0001 C CNN
-F 3 "" H 3800 4025 50  0001 C CNN
-	1    3800 4025
+P 3050 4125
+F 0 "#PWR0106" H 3050 3875 50  0001 C CNN
+F 1 "GND" H 3055 3952 50  0000 C CNN
+F 2 "" H 3050 4125 50  0001 C CNN
+F 3 "" H 3050 4125 50  0001 C CNN
+	1    3050 4125
 	1    0    0    -1
 $EndComp
@@
 L power:VCC #PWR0107
 U 1 1 5F7AB9A0
-P 3800 3600
-F 0 "#PWR0107" H 3800 3450 50  0001 C CNN
-F 1 "VCC" H 3815 3773 50  0000 C CNN
-F 2 "" H 3800 3600 50  0001 C CNN
-F 3 "" H 3800 3600 50  0001 C CNN
-	1    3800 3600
-	1    0    0    -1
-$EndComp
-Wire Wire Line
-	3800 3600 3800 3775
-Wire Wire Line
-	3800 3775 3600 3775
-Wire Wire Line
-	3600 3825 3800 3825
-Wire Wire Line
-	3800 3825 3800 4025
-NoConn ~ 3600 3725
+P 3050 3700
+F 0 "#PWR0107" H 3050 3550 50  0001 C CNN
+F 1 "VCC" H 3065 3873 50  0000 C CNN
+F 2 "" H 3050 3700 50  0001 C CNN
+F 3 "" H 3050 3700 50  0001 C CNN
+	1    3050 3700
+	1    0    0    -1
+$EndComp
+Wire Wire Line
+	3050 3700 3050 3875
+Wire Wire Line
+	3050 3875 2850 3875
+Wire Wire Line
+	2850 3925 3050 3925
+Wire Wire Line
+	3050 3925 3050 4125
+NoConn ~ 2850 3825
 Text GLabel 2050 5400 2    50   Input ~ 0
 F6
@@
 L Mechanical:MountingHole_Pad GND1
 U 1 1 5F8A75FD
-P 5650 7150
-F 0 "GND1" V 5604 7300 50  0000 L CNN
-F 1 "MountingHole_Pad" V 5695 7300 50  0000 L CNN
-F 2 "foostan:1pin_conn" H 5650 7150 50  0001 C CNN
-F 3 "~" H 5650 7150 50  0001 C CNN
-	1    5650 7150
+P 5650 6950
+F 0 "GND1" V 5604 7100 50  0000 L CNN
+F 1 "MountingHole_Pad" V 5695 7100 50  0000 L CNN
+F 2 "foostan:1pin_conn" H 5650 6950 50  0001 C CNN
+F 3 "~" H 5650 6950 50  0001 C CNN
+	1    5650 6950
 	0    1    1    0
 $EndComp
@@
 $EndComp
 Wire Wire Line
-	3600 3875 3925 3875
-Text GLabel 3925 3875 2    50   Input ~ 0
+	2850 3975 3175 3975
+Text GLabel 3175 3975 2    50   Input ~ 0
 data
 Text GLabel 5050 6550 0    50   Input ~ 0
@@
 	5550 6150 5050 6150
 Wire Wire Line
-	5550 7150 5050 7150
+	5550 6950 5050 6950
 $Comp
 L power:GND #PWR04
 U 1 1 5F995F04
-P 5050 7150
-F 0 "#PWR04" H 5050 6900 50  0001 C CNN
-F 1 "GND" H 5055 6977 50  0000 C CNN
-F 2 "" H 5050 7150 50  0001 C CNN
-F 3 "" H 5050 7150 50  0001 C CNN
-	1    5050 7150
+P 5050 6950
+F 0 "#PWR04" H 5050 6700 50  0001 C CNN
+F 1 "GND" H 5055 6777 50  0000 C CNN
+F 2 "" H 5050 6950 50  0001 C CNN
+F 3 "" H 5050 6950 50  0001 C CNN
+	1    5050 6950
 	1    0    0    -1
 $EndComp
@@
 Connection ~ 8150 3400
 Connection ~ 7450 3400
-Wire Wire Line
-	5050 6950 5550 6950
-Text GLabel 5050 6950 0    50   Input ~ 0
+Text GLabel 4300 5000 0    50   Input ~ 0
 B5
-$Comp
-L Mechanical:MountingHole_Pad B5
-U 1 1 6008F413
-P 5650 6950
-F 0 "B5" V 5696 7099 50  0000 L CNN
-F 1 "MountingHole_Pad" V 5605 7099 50  0000 L CNN
-F 2 "foostan:1pin_conn" H 5650 6950 50  0001 C CNN
-F 3 "~" H 5650 6950 50  0001 C CNN
-	1    5650 6950
-	0    1    -1   0
-$EndComp
 Wire Wire Line
 	5450 2150 5450 3100
@@
 L power:VCC #PWR06
 U 1 1 601CCD3A
-P 4600 5000
-F 0 "#PWR06" H 4600 4850 50  0001 C CNN
-F 1 "VCC" H 4615 5173 50  0000 C CNN
-F 2 "" H 4600 5000 50  0001 C CNN
-F 3 "" H 4600 5000 50  0001 C CNN
-	1    4600 5000
+P 4300 3800
+F 0 "#PWR06" H 4300 3650 50  0001 C CNN
+F 1 "VCC" H 4315 3973 50  0000 C CNN
+F 2 "" H 4300 3800 50  0001 C CNN
+F 3 "" H 4300 3800 50  0001 C CNN
+	1    4300 3800
+	1    0    0    -1
+$EndComp
+Text GLabel 4300 4000 0    50   Input ~ 0
+F5
+Text GLabel 4300 3900 0    50   Input ~ 0
+F4
+$Comp
+L power:GND #PWR07
+U 1 1 601D9867
+P 4300 4100
+F 0 "#PWR07" H 4300 3850 50  0001 C CNN
+F 1 "GND" H 4305 3927 50  0000 C CNN
+F 2 "" H 4300 4100 50  0001 C CNN
+F 3 "" H 4300 4100 50  0001 C CNN
+	1    4300 4100
 	1    0    0    -1
 $EndComp
@@
 L local:joystick U2
 U 1 1 601D4158
-P 4900 5150
-F 0 "U2" H 5128 5201 50  0000 L CNN
-F 1 "joystick" H 5128 5110 50  0000 L CNN
-F 2 "local:J08K" H 4900 4850 50  0001 C CNN
-F 3 "" H 4900 4850 50  0001 C CNN
-	1    4900 5150
-	1    0    0    -1
-$EndComp
-$Comp
-L power:GND #PWR07
-U 1 1 601D9867
-P 4600 5300
-F 0 "#PWR07" H 4600 5050 50  0001 C CNN
-F 1 "GND" H 4605 5127 50  0000 C CNN
-F 2 "" H 4600 5300 50  0001 C CNN
-F 3 "" H 4600 5300 50  0001 C CNN
-	1    4600 5300
-	1    0    0    -1
-$EndComp
-Text GLabel 4600 5100 0    50   Input ~ 0
+P 4600 3950
+F 0 "U2" H 4828 4001 50  0000 L CNN
+F 1 "joystick" H 4828 3910 50  0000 L CNN
+F 2 "local:J08K" H 4600 3650 50  0001 C CNN
+F 3 "" H 4600 3650 50  0001 C CNN
+	1    4600 3950
+	1    0    0    -1
+$EndComp
+$Comp
+L local:joystick_s U3
+U 1 1 604A6B52
+P 4600 5000
+F 0 "U3" H 4828 5051 50  0000 L CNN
+F 1 "joystick_s" H 4828 4960 50  0000 L CNN
+F 2 "local:Joycon_Stick" H 4600 4700 50  0001 C CNN
+F 3 "" H 4600 4700 50  0001 C CNN
+	1    4600 5000
+	1    0    0    -1
+$EndComp
+Text GLabel 4300 5200 0    50   Input ~ 0
 F4
-Text GLabel 4600 5200 0    50   Input ~ 0
+Text GLabel 4300 4900 0    50   Input ~ 0
 F5
+$Comp
+L power:VCC #PWR0108
+U 1 1 604BCAF5
+P 4300 4800
+F 0 "#PWR0108" H 4300 4650 50  0001 C CNN
+F 1 "VCC" H 4315 4973 50  0000 C CNN
+F 2 "" H 4300 4800 50  0001 C CNN
+F 3 "" H 4300 4800 50  0001 C CNN
+	1    4300 4800
+	1    0    0    -1
+$EndComp
+$Comp
+L power:GND #PWR0109
+U 1 1 604D24B1
+P 4050 5100
+F 0 "#PWR0109" H 4050 4850 50  0001 C CNN
+F 1 "GND" H 4055 4927 50  0000 C CNN
+F 2 "" H 4050 5100 50  0001 C CNN
+F 3 "" H 4050 5100 50  0001 C CNN
+	1    4050 5100
+	1    0    0    -1
+$EndComp
+Wire Wire Line
+	4300 5100 4050 5100
+$Comp
+L Device:Jumper JP_NOJS1
+U 1 1 604EEF7A
+P 3000 7000
+F 0 "JP_NOJS1" H 3000 6868 50  0000 C CNN
+F 1 "Jumper" H 3000 6777 50  0000 C CNN
+F 2 "Jumper:SolderJumper-2_P1.3mm_Open_RoundedPad1.0x1.5mm" H 3000 7000 50  0001 C CNN
+F 3 "~" H 3000 7000 50  0001 C CNN
+	1    3000 7000
+	1    0    0    -1
+$EndComp
+$Comp
+L power:GND #PWR0110
+U 1 1 604EF580
+P 3300 7000
+F 0 "#PWR0110" H 3300 6750 50  0001 C CNN
+F 1 "GND" H 3305 6827 50  0000 C CNN
+F 2 "" H 3300 7000 50  0001 C CNN
+F 3 "" H 3300 7000 50  0001 C CNN
+	1    3300 7000
+	1    0    0    -1
+$EndComp
+Text GLabel 2700 7000 0    50   Input ~ 0
+B5
 $EndSCHEMATC

Commit message: update musashi50.sch
Parts:
- removed U2: joystick, local:J08K, symbol local:joystick
- added D_E5, D_F1: D, foostan:D3_TH_SMD, symbol Device:D
- added SW_E5, SW_F1: SW_PUSH, local:CherryMX_Direct_Hotswap_Reversible, symbol foostan:SW_PUSH
Connections:
- wire segments 86 -> 90
Changed lines of the file:
@@
 Connection ~ 8150 3400
 Connection ~ 7450 3400
-Text GLabel 4300 5000 0    50   Input ~ 0
+Text GLabel 4250 3900 0    50   Input ~ 0
 B5
 Wire Wire Line
-	5450 2150 5450 3100
+	5450 2150 5450 2450
 Wire Wire Line
 	6150 2150 6150 2450
@@
 Connection ~ 6750 3400
 $Comp
-L power:VCC #PWR06
-U 1 1 601CCD3A
-P 4300 3800
-F 0 "#PWR06" H 4300 3650 50  0001 C CNN
-F 1 "VCC" H 4315 3973 50  0000 C CNN
-F 2 "" H 4300 3800 50  0001 C CNN
-F 3 "" H 4300 3800 50  0001 C CNN
-	1    4300 3800
+L local:joystick_s U3
+U 1 1 604A6B52
+P 4550 3900
+F 0 "U3" H 4778 3951 50  0000 L CNN
+F 1 "joystick_s" H 4778 3860 50  0000 L CNN
+F 2 "local:Joycon_Stick" H 4550 3600 50  0001 C CNN
+F 3 "" H 4550 3600 50  0001 C CNN
+	1    4550 3900
 	1    0    0    -1
 $EndComp
-Text GLabel 4300 4000 0    50   Input ~ 0
-F5
-Text GLabel 4300 3900 0    50   Input ~ 0
+Text GLabel 4250 4100 0    50   Input ~ 0
 F4
-$Comp
-L power:GND #PWR07
-U 1 1 601D9867
-P 4300 4100
-F 0 "#PWR07" H 4300 3850 50  0001 C CNN
-F 1 "GND" H 4305 3927 50  0000 C CNN
-F 2 "" H 4300 4100 50  0001 C CNN
-F 3 "" H 4300 4100 50  0001 C CNN
-	1    4300 4100
-	1    0    0    -1
-$EndComp
-$Comp
-L local:joystick U2
-U 1 1 601D4158
-P 4600 3950
-F 0 "U2" H 4828 4001 50  0000 L CNN
-F 1 "joystick" H 4828 3910 50  0000 L CNN
-F 2 "local:J08K" H 4600 3650 50  0001 C CNN
-F 3 "" H 4600 3650 50  0001 C CNN
-	1    4600 3950
-	1    0    0    -1
-$EndComp
-$Comp
-L local:joystick_s U3
-U 1 1 604A6B52
-P 4600 5000
-F 0 "U3" H 4828 5051 50  0000 L CNN
-F 1 "joystick_s" H 4828 4960 50  0000 L CNN
-F 2 "local:Joycon_Stick" H 4600 4700 50  0001 C CNN
-F 3 "" H 4600 4700 50  0001 C CNN
-	1    4600 5000
-	1    0    0    -1
-$EndComp
-Text GLabel 4300 5200 0    50   Input ~ 0
-F4
-Text GLabel 4300 4900 0    50   Input ~ 0
+Text GLabel 4250 3800 0    50   Input ~ 0
 F5
 $Comp
 L power:VCC #PWR0108
 U 1 1 604BCAF5
-P 4300 4800
-F 0 "#PWR0108" H 4300 4650 50  0001 C CNN
-F 1 "VCC" H 4315 4973 50  0000 C CNN
-F 2 "" H 4300 4800 50  0001 C CNN
-F 3 "" H 4300 4800 50  0001 C CNN
-	1    4300 4800
+P 4250 3700
+F 0 "#PWR0108" H 4250 3550 50  0001 C CNN
+F 1 "VCC" H 4265 3873 50  0000 C CNN
+F 2 "" H 4250 3700 50  0001 C CNN
+F 3 "" H 4250 3700 50  0001 C CNN
+	1    4250 3700
 	1    0    0    -1
 $EndComp
@@
 L power:GND #PWR0109
 U 1 1 604D24B1
-P 4050 5100
-F 0 "#PWR0109" H 4050 4850 50  0001 C CNN
-F 1 "GND" H 4055 4927 50  0000 C CNN
-F 2 "" H 4050 5100 50  0001 C CNN
-F 3 "" H 4050 5100 50  0001 C CNN
-	1    4050 5100
+P 4000 4000
+F 0 "#PWR0109" H 4000 3750 50  0001 C CNN
+F 1 "GND" H 4005 3827 50  0000 C CNN
+F 2 "" H 4000 4000 50  0001 C CNN
+F 3 "" H 4000 4000 50  0001 C CNN
+	1    4000 4000
 	1    0    0    -1
 $EndComp
 Wire Wire Line
-	4300 5100 4050 5100
+	4250 4000 4000 4000
 $Comp
 L Device:Jumper JP_NOJS1
@@
 Text GLabel 2700 7000 0    50   Input ~ 0
 B5
+$Comp
+L foostan:SW_PUSH SW_F1
+U 1 1 605FBDAB
+P 5750 2450
+F 0 "SW_F1" H 5750 2705 50  0000 C CNN
+F 1 "SW_PUSH" H 5750 2614 50  0000 C CNN
+F 2 "local:CherryMX_Direct_Hotswap_Reversible" H 5750 2450 50  0001 C CNN
+F 3 "" H 5750 2450 50  0000 C CNN
+	1    5750 2450
+	1    0    0    -1
+$EndComp
+Connection ~ 5450 2450
+Wire Wire Line
+	5450 2450 5450 3100
+$Comp
+L Device:D D_F1
+U 1 1 605FD473
+P 6050 2600
+F 0 "D_F1" V 6096 2680 50  0000 L CNN
+F 1 "D" V 6005 2680 50  0000 L CNN
+F 2 "foostan:D3_TH_SMD" H 6050 2600 50  0001 C CNN
+F 3 "~" H 6050 2600 50  0001 C CNN
+	1    6050 2600
+	0    -1   -1   0
+$EndComp
+Wire Wire Line
+	6750 2750 6050 2750
+Connection ~ 6750 2750
+$Comp
+L foostan:SW_PUSH SW_E5
+U 1 1 6060C4D7
+P 6450 5050
+F 0 "SW_E5" H 6450 5305 50  0000 C CNN
+F 1 "SW_PUSH" H 6450 5214 50  0000 C CNN
+F 2 "local:CherryMX_Direct_Hotswap_Reversible" H 6450 5050 50  0001 C CNN
+F 3 "" H 6450 5050 50  0000 C CNN
+	1    6450 5050
+	1    0    0    -1
+$EndComp
+Wire Wire Line
+	6150 4400 6150 5050
+Connection ~ 6150 4400
+$Comp
+L Device:D D_E5
+U 1 1 60616038
+P 6750 5200
+F 0 "D_E5" V 6796 5280 50  0000 L CNN
+F 1 "D" V 6705 5280 50  0000 L CNN
+F 2 "foostan:D3_TH_SMD" H 6750 5200 50  0001 C CNN
+F 3 "~" H 6750 5200 50  0001 C CNN
+	1    6750 5200
+	0    -1   -1   0
+$EndComp
+Wire Wire Line
+	7450 5350 6750 5350
+Connection ~ 7450 5350
 $EndSCHEMATC
