File: pcb/musashi60-revD.kicad_pcb (KiCad board)
At the start: 2 copper layers, 160 x 135 mm, 68 parts, among them J1 MJ-4PP-9, U1 ProMicro_r

Commit message: update revD pcb
Parts:
- JP_LEFT1, JP_RIGHT1: footprint Jumper:SolderJumper-2_P1.3mm_Open_RoundedPad1.0x1.5mm -> local:SolderJumper
- OL1: value OLED_Reversible -> OLED
- SW_RST1: footprint foostan:ResetSW -> local:ResetSW
- moved OL1 5.82 mm to (171.6, 89.6)
- moved J1 3.00 mm to (188.0, 75.0)
- moved SW_RST1 3.00 mm to (169.0, 74.0), turned to 180 degrees
- moved SW_A5 2.60 mm to (167.8, 146.0)
- moved JP_LEFT1 2.53 mm to (154.0, 48.0), turned to 0 degrees
- moved JP_RIGHT1 2.53 mm to (154.0, 48.0), turned to 180 degrees
- moved U1 2.50 mm to (169.0, 51.6)
- moved D_A5 2.42 mm to (161.6, 151.6)
- moved D_A3 2.20 mm to (151.6, 107.4), turned to 175 degrees
- moved SW_D5 1.90 mm to (101.7, 119.3)
- moved D_D5 1.90 mm to (101.6, 127.6)
- moved D_B1 1.81 mm to (137.0, 53.0)
- moved D_B4 1.81 mm to (132.4, 109.8)
- moved SW_B3 1.81 mm to (134.6, 83.0)
- moved SW_B4 1.81 mm to (133.0, 101.7)
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Other:
- board size 160 x 135 mm -> 163 x 135 mm

Commit message: update scheme for revD
Parts:
- removed G_LOGO_B, G_LOGO_F: LOGO, local:musashi60-silk-384
- added G***: LOGO, local:musashi60-silk-384, B.Cu at (68.9, 123.2)
- added G***: LOGO, local:musashi60-silk-384, F.Cu at (68.7, 123.1)
- added U2: OLED_Reversible_Jumper, local:OLED_Reversible_Jumper, F.Cu at (171.4, 82.7)
- D_A2, D_A3, D_A5, D_B1, D_B2, D_B3, D_B4, D_B5, D_C1, D_C2, D_C3, D_C4, D_C5, D_D1, D_D2, D_D3, D_D4, D_D5, D_E1, D_E2, D_E3, D_E4, D_F1, D_F2, D_F3, D_F4, D_G1, D_G2, D_G3, D_G4: footprint foostan:D3_TH_SMD -> local:D_TH
- moved OL1 12.5 mm to (171.3, 102.1), turned to 0 degrees
- moved D_A5 3.76 mm to (163.2, 148.2), turned to 140 degrees
- moved SW_A5 3.73 mm to (169.1, 142.5), turned to 140 degrees
- moved SW_B5 1.90 mm to (150.9, 129.8), turned to 150 degrees
- moved D_B5 1.60 mm to (146.4, 136.7), turned to 150 degrees
- moved D_C5 0.71 mm to (124.9, 128.9)
- moved SW_C5 0.71 mm to (126.5, 120.8)
- moved SW_D5 0.67 mm to (101.1, 119.6), turned to 185 degrees
- moved SW_A2 0.41 mm to (154.5, 75.7)
- moved D_A2 0.41 mm to (153.4, 83.8)
- moved D_F2 0.40 mm to (54.1, 70.4)
- moved D_F4 0.34 mm to (56.0, 110.7)
- moved SW_F4 0.34 mm to (55.7, 102.6)
- moved SW_A3 0.32 mm to (152.3, 99.5)
- moved D_A3 0.32 mm to (151.7, 107.7)
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Connections:
- OL1 pad 1: D1 -> Net-(OL1-Pad1)
- OL1 pad 2: D0 -> Net-(OL1-Pad2)
- OL1 pad 3: VCC -> Net-(OL1-Pad3)
- OL1 pad 4: GND -> Net-(OL1-Pad4)
Other:
- board size 163 x 135 mm -> 163 x 130 mm
