File: pcb/revG/revG-thumb.kicad_pcb (KiCad board)
At the start: 2 copper layers, 78 x 33 mm, 14 parts

Commit message: update revG-thumb.kicad_pcb
Parts:
- D_LD5: value D_C5 -> D_D5
- H_L5, H_LA1, H_LB1, H_LC1, H_LD5, H_LGND1: footprint local:Pin_D0.7mm -> local:Pin_D0.8mm
- moved D_LD5 0.50 mm to (39.0, 47.0)
